File: Mechatronics/Hardware/Electrical/BEncoderBoard/EncoderBoard.sch (KiCad schematic (older format))
At the start: 32 parts, among them J1 Conn_01x01_Male, J10 Conn_01x01_Male, J2 Conn_01x01_Male, J3 Conn_01x01_Male, J4 Conn_01x01_Male, J5 Conn_01x01_Male, J6 Conn_01x01_Male, J7 Conn_01x01_Male, J8 Conn_01x01_Male, J9 Conn_01x01_Male, Q1 Q_NMOS_SGD, Q2 Q_NMOS_SGD, Q3 Q_NMOS_SGD, U1 ATmega328-PU, U2 ITR1802A, U3 ITR1802B, U4 HEF40106BT, Y1 20Mhz

Commit message: Changes
Parts:
- removed C1, C2: .1uF, Encoder:C_Disc_D9.0mm_W5.0mm_P5.00mm, symbol Device:C
- removed C3, C4: 22pF, Encoder:C_Disc_D9.0mm_W5.0mm_P5.00mm, symbol Device:C
- removed J1, J3, J4, J5: Conn_01x01_Male, Encoder:PinHeader_1x01_P2.54mm_Vertical, symbol Connector:Conn_01x01_Male
- removed Q1, Q2, Q3: Q_NMOS_SGD, Encoder:TO-92_Inline_Wide, symbol Device:Q_NMOS_SGD
- removed R10, R5, R6, R7, R8, R9: 10K, Encoder:R_Axial_DIN0414_L11.9mm_D4.5mm_P15.24mm_Horizontal, symbol Device:R
- removed U1: ATmega328-PU, Encoder:DIP-28_W7.62mm_LongPads, symbol MCU_Microchip_ATmega:ATmega328-PU
- removed U4: HEF40106BT, Encoder:SOIC-14, symbol Encoder:HEF40106BT
- removed Y1: 20Mhz, Encoder:Crystal_HC49-U_Vertical, symbol Device:Crystal
- added C? (x2): 12pF, symbol Device:C
- added C? (x7): 100nF, symbol Device:C
- added C?: 10uF, Encoder:C_Disc_D9.0mm_W5.0mm_P5.00mm, symbol Device:C
- added C?: .1uF, Encoder:C_Disc_D9.0mm_W5.0mm_P5.00mm, symbol Device:C
- added C?: 4.7uF, symbol Device:C
- added C?: 10uF, symbol Device:C
- added C?: 1uF, symbol Device:C
- added D? (x2): TVS, Encoder:D_DO-201AD_P15.24mm_Horizontal, symbol Device:D_Zener
- added D?: D_Schottky, Encoder:D_DO-201AD_P15.24mm_Horizontal, symbol Device:D_Schottky
- added IC?: RN4020-V_RM120, RN4020-V/RM123, symbol Encoder:RN4020-V_RM120
- added J? (x13): Conn_01x01_Male, Encoder:PinHeader_1x01_P2.54mm_Vertical, symbol Connector:Conn_01x01_Male
- added Q?: Q_PMOS_GDS, Encoder:TO-220-3_Horizontal_TabDown, symbol Device:Q_PMOS_GDS
- added R?: 10K, Encoder:R_Axial_DIN0414_L11.9mm_D4.5mm_P15.24mm_Horizontal, symbol Device:R
- added R?: 10K, symbol Device:R
- added S?: EG1218, Encoder:Switch_Slide_11.6x4mm_EG1218, symbol Encoder:EG1218
- added U?: STM32F103C8T6, QFP50P900X900X160-48N, symbol Encoder:STM32F103C8T6
- added U?: LD1117S33TR_SOT223, Encoder:TO-220-3_Horizontal_TabDown, symbol Regulator_Linear:LD1117S33TR_SOT223
- added U?: MT3608A, Encoder:Mt3608, symbol Encoder:MT3608A
- added U?: 03962A, Encoder:03962A, symbol Encoder:03962A
- added U?: SSD1306OLED, symbol Encoder:SSD1306OLED
- added Y?: 8Mhz, symbol Device:Crystal
Connections:
- net labels added: F1RX, F1SCL, F1SDA, F1TX, SWCLK, SWDIO, SensorsEnable, VCC
- net labels removed: 3VCMD, 3VRX, 3VTX, OUTA, OUTB, RX, TX
- wire segments 83 -> 134
- no-connect marks 21 -> 16
Other:
- moved on the sheet: J10, J2, J6, J7, J8, J9, R1, R2, R3, R4, U2, U3

Commit message: Changes
Parts:
- removed C?: 10uF, Encoder:C_Disc_D9.0mm_W5.0mm_P5.00mm, symbol Device:C
- removed C?: .1uF, Encoder:C_Disc_D9.0mm_W5.0mm_P5.00mm, symbol Device:C
- removed D?: TVS, Encoder:D_DO-201AD_P15.24mm_Horizontal, symbol Device:D_Zener
- removed J7, J8, J? (x5): Conn_01x01_Male, Encoder:PinHeader_1x01_P2.54mm_Vertical, symbol Connector:Conn_01x01_Male
- removed U?: LD1117S33TR_SOT223, Encoder:TO-220-3_Horizontal_TabDown, symbol Regulator_Linear:LD1117S33TR_SOT223
- removed U?: MT3608A, Encoder:Mt3608, symbol Encoder:MT3608A
- added C? (x2): 1uF, symbol Device:C
- added C?: 4.7uF, symbol Device:C
- added R?: 10K, symbol Device:R
- added U?: LTC2430, symbol Encoder:LTC2430
Connections:
- net labels added: Batt+, Batt-
- net labels removed: +5V, SCL, SDA
- wire segments 134 -> 121
Other:
- moved on the sheet: D?, J?, R?

Commit message: Changes
Parts:
- removed C?: 100nF, symbol Device:C
- removed J10, J2, J6, J9, J? (x8): Conn_01x01_Male, Encoder:PinHeader_1x01_P2.54mm_Vertical, symbol Connector:Conn_01x01_Male
- removed Q?: Q_PMOS_GDS, Encoder:TO-220-3_Horizontal_TabDown, symbol Device:Q_PMOS_GDS
- removed U?: 03962A, Encoder:03962A, symbol Encoder:03962A
- added C13: 10uF, Encoder:C_0603_1608Metric_Pad1.05x0.95mm_HandSolder, symbol Device:C
- added C16: .1uF, Encoder:C_0603_1608Metric_Pad1.05x0.95mm_HandSolder, symbol Device:C
- added IC2: TP4056, Encoder:Sop(8), symbol Encoder:TP4056
- added IC3: DW01+G, Encoder:Sot-23(6), symbol Encoder:DW01+G
- added J1: Conn_01x07_Male, Encoder:PinSocket_1x07_P2.54mm_Vertical, symbol Connector:Conn_01x07_Male
- added J4: Barrel_Jack_Switch, Encoder:BarrelJack_Horizontal, symbol Connector:Barrel_Jack_Switch
- added J5: Batt+, Encoder:PinHeader_1x01_P2.54mm_Vertical, symbol Connector:Conn_01x01_Male
- added J7: Batt-, Encoder:PinHeader_1x01_P2.54mm_Vertical, symbol Connector:Conn_01x01_Male
- added Q1: FS8205, Encoder:Sot-23(6), symbol Encoder:FS8205
- added Q2: Q_PMOS_GSD, symbol Encoder:Q_PMOS_GSD
- added R11: 100, Encoder:R_0603_1608Metric_Pad1.05x0.95mm_HandSolder, symbol Device:R
- added R13, R14: 10K, Encoder:R_0603_1608Metric_Pad1.05x0.95mm_HandSolder, symbol Device:R
- added R8: 1.2K, Encoder:R_0603_1608Metric_Pad1.05x0.95mm_HandSolder, symbol Device:R
- added R9: 1K, Encoder:R_0603_1608Metric_Pad1.05x0.95mm_HandSolder, symbol Device:R
- C1, C10, C11, C12, C14, C15, C2, C3, C4, C5, C6, C7, C8, C9: renamed from C?; footprint (none) -> Encoder:C_0603_1608Metric_Pad1.05x0.95mm_HandSolder
- IC1: renamed from IC?; footprint RN4020-V/RM123 -> Encoder:Bluetooth_Module_RN4020
- R1, R2, R3, R4: footprint Encoder:R_Axial_DIN0414_L11.9mm_D4.5mm_P15.24mm_Horizontal -> Encoder:R_0603_1608Metric_Pad1.05x0.95mm_HandSolder
- R5, R7: renamed from R?; footprint (none) -> Encoder:R_0603_1608Metric_Pad1.05x0.95mm_HandSolder
- R6: renamed from R?; footprint Encoder:R_Axial_DIN0414_L11.9mm_D4.5mm_P15.24mm_Horizontal -> Encoder:R_0603_1608Metric_Pad1.05x0.95mm_HandSolder
- U1: renamed from U?; footprint QFP50P900X900X160-48N -> Encoder:QFP50P900X900X160-48N
- U5: renamed from U?; footprint (none) -> Encoder:PinSocket_1x04_P2.54mm_Vertical
- U6: renamed from U?; footprint (none) -> Encoder:DFN-6_DC
- Y1: renamed from Y?; footprint (none) -> Encoder:Crystal_HC49-U_Vertical
- gave numbers to parts that had none: 3
Connections:
- net labels added: BattVolt, CHG, CTS, RTS, STDBY
- net labels removed: Batt+, Batt-, BattVoltSens, CMD, PowSupStat, SensorsEnable
- wire segments 121 -> 168
- no-connect marks 16 -> 34
Other:
- moved on the sheet: C1, C10, C11, C12, C14, C15, C2, C3, C4, C5, C6, C7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

Commit message: Added changes
Parts:
- removed D1: TVS, Encoder:D_DO-201AD_P15.24mm_Horizontal, symbol Device:D_Zener
- removed D2: D_Schottky, Encoder:D_DO-201AD_P15.24mm_Horizontal, symbol Device:D_Schottky
- added D1: D, Encoder:D_SMA, symbol Device:D
- J5, J7: footprint Encoder:PinHeader_1x01_P2.54mm_Vertical -> Encoder:No3dmodelPinHeader_1x01_P2.54mm_Vertical
- Q2: footprint (none) -> Encoder:SOT-23
Connections:
- wire segments 168 -> 167
- no-connect marks 34 -> 36
Changed lines of the file:
@@
 Wire Wire Line
 	5650 6750 5650 6900
-$Comp
-L Device:D_Zener D1
-U 1 1 5D40B7CD
-P 2100 5850
-F 0 "D1" V 2054 5929 50  0000 L CNN
-F 1 "TVS" V 2145 5929 50  0000 L CNN
-F 2 "Encoder:D_DO-201AD_P15.24mm_Horizontal" H 2100 5850 50  0001 C CNN
-F 3 "~" H 2100 5850 50  0001 C CNN
-	1    2100 5850
-	0    1    1    0
-$EndComp
 Connection ~ 6450 5700
 Wire Wire Line
@@
 $EndComp
 $Comp
-L Device:D_Schottky D2
-U 1 1 5D40B8AB
-P 6750 5950
-F 0 "D2" V 6796 5871 50  0000 R CNN
-F 1 "D_Schottky" V 6705 5871 50  0000 R CNN
-F 2 "Encoder:D_DO-201AD_P15.24mm_Horizontal" H 6750 5950 50  0001 C CNN
-F 3 "~" H 6750 5950 50  0001 C CNN
-	1    6750 5950
-	0    -1   -1   0
-$EndComp
-$Comp
 L Encoder:LTC2430 U6
 U 1 1 5D41A14E
@@
 Wire Wire Line
 	6750 5700 7300 5700
-Wire Wire Line
-	6750 6100 6750 6750
 Wire Wire Line
 	7900 6650 7900 5950
@@
 F 0 "J7" H 5873 7780 50  0000 R CNN
 F 1 "Batt-" H 5873 7871 50  0000 R CNN
-F 2 "Encoder:PinHeader_1x01_P2.54mm_Vertical" H 5900 7850 50  0001 C CNN
+F 2 "Encoder:No3dmodelPinHeader_1x01_P2.54mm_Vertical" H 5900 7850 50  0001 C CNN
 F 3 "~" H 5900 7850 50  0001 C CNN
 	1    5900 7850
@@
 F 0 "J5" H 5823 6480 50  0000 R CNN
 F 1 "Batt+" H 5823 6571 50  0000 R CNN
-F 2 "Encoder:PinHeader_1x01_P2.54mm_Vertical" H 5850 6550 50  0001 C CNN
+F 2 "Encoder:No3dmodelPinHeader_1x01_P2.54mm_Vertical" H 5850 6550 50  0001 C CNN
 F 3 "~" H 5850 6550 50  0001 C CNN
 	1    5850 6550
@@
 Wire Wire Line
 	1800 5450 1800 5700
-Wire Wire Line
-	1800 5700 2100 5700
-Connection ~ 2100 5700
-$Comp
-L power:GND #PWR06
-U 1 1 5D706B3B
-P 2100 6000
-F 0 "#PWR06" H 2100 5750 50  0001 C CNN
-F 1 "GND" H 2105 5827 50  0000 C CNN
-F 2 "" H 2100 6000 50  0001 C CNN
-F 3 "" H 2100 6000 50  0001 C CNN
-	1    2100 6000
-	1    0    0    -1
-$EndComp
 Connection ~ 1800 5700
 $Comp
@@
 Wire Wire Line
 	1700 900  2150 900
-Wire Wire Line
-	2100 5700 2550 5700
 Wire Wire Line
 	5000 5700 6450 5700
@@
 F 0 "Q2" H 6450 6500 50  0000 C CNN
 F 1 "Q_PMOS_GSD" H 6450 6409 50  0000 C CNN
-F 2 "" V 6650 6550 50  0001 C CNN
+F 2 "Encoder:SOT-23" V 6650 6550 50  0001 C CNN
 F 3 "~" V 6450 6750 50  0001 C CNN
 	1    6450 6700
 	1    0    0    -1
 $EndComp
+Wire Wire Line
+	1800 5700 2550 5700
+$Comp
+L Device:D D1
+U 1 1 5D4F6601
+P 6750 5950
+F 0 "D1" V 6796 5871 50  0000 R CNN
+F 1 "D" V 6705 5871 50  0000 R CNN
+F 2 "Encoder:D_SMA" H 6750 5950 50  0001 C CNN
+F 3 "~" H 6750 5950 50  0001 C CNN
+	1    6750 5950
+	0    -1   -1   0
+$EndComp
+Wire Wire Line
+	6750 6100 6750 6750
+NoConn ~ 3850 8650
+NoConn ~ 5050 8650
 $EndSCHEMATC

Commit message: Added changes
Connections:
- net labels added: BOOT0
- no-connect marks 36 -> 37
Other:
- moved on the sheet: R13, R14
Changed lines of the file:
@@
 	2150 900  3200 900
-Wire Wire Line
-	750  900  1700 900
 Wire Wire Line
 	4450 3050 6900 3050
@@
 NoConn ~ 4450 2450
 NoConn ~ 4450 2650
-NoConn ~ 4450 2750
 Wire Wire Line
 	4450 3450 5100 3450
-Text Label 2000 2350 0    50   ~ 0
-BattVolt
 Text Label 4650 3450 0    50   ~ 0
 CHG
-Wire Wire Line
-	4450 3350 7400 3350
-Wire Wire Line
-	7400 3050 7750 3050
-Wire Wire Line
-	7400 3050 7400 3350
 NoConn ~ 7750 3150
 Wire Wire Line
@@
 L Device:R R13
 U 1 1 5D7ED20E
-P 1700 1550
-F 0 "R13" H 1770 1596 50  0000 L CNN
-F 1 "10K" H 1770 1505 50  0000 L CNN
-F 2 "Encoder:R_0603_1608Metric_Pad1.05x0.95mm_HandSolder" V 1630 1550 50  0001 C CNN
-F 3 "~" H 1700 1550 50  0001 C CNN
-	1    1700 1550
+P 1700 2550
+F 0 "R13" H 1770 2596 50  0000 L CNN
+F 1 "10K" H 1770 2505 50  0000 L CNN
+F 2 "Encoder:R_0603_1608Metric_Pad1.05x0.95mm_HandSolder" V 1630 2550 50  0001 C CNN
+F 3 "~" H 1700 2550 50  0001 C CNN
+	1    1700 2550
 	1    0    0    -1
 $EndComp
@@
 L Device:R R14
 U 1 1 5D7ED33E
-P 1700 2500
-F 0 "R14" H 1770 2546 50  0000 L CNN
-F 1 "10K" H 1770 2455 50  0000 L CNN
-F 2 "Encoder:R_0603_1608Metric_Pad1.05x0.95mm_HandSolder" V 1630 2500 50  0001 C CNN
-F 3 "~" H 1700 2500 50  0001 C CNN
-	1    1700 2500
+P 1700 2850
+F 0 "R14" H 1770 2896 50  0000 L CNN
+F 1 "10K" H 1770 2805 50  0000 L CNN
+F 2 "Encoder:R_0603_1608Metric_Pad1.05x0.95mm_HandSolder" V 1630 2850 50  0001 C CNN
+F 3 "~" H 1700 2850 50  0001 C CNN
+	1    1700 2850
 	1    0    0    -1
 $EndComp
@@
 L power:GND #PWR038
 U 1 1 5D7ED632
-P 1700 2650
-F 0 "#PWR038" H 1700 2400 50  0001 C CNN
-F 1 "GND" H 1705 2477 50  0000 C CNN
-F 2 "" H 1700 2650 50  0001 C CNN
-F 3 "" H 1700 2650 50  0001 C CNN
-	1    1700 2650
-	1    0    0    -1
-$EndComp
-Wire Wire Line
-	1700 2350 2450 2350
-Wire Wire Line
-	1700 2350 1700 1700
-Connection ~ 1700 2350
-Wire Wire Line
-	1700 1400 1700 900
-Connection ~ 1700 900
-Wire Wire Line
-	1700 900  2150 900
+P 1700 3000
+F 0 "#PWR038" H 1700 2750 50  0001 C CNN
+F 1 "GND" H 1705 2827 50  0000 C CNN
+F 2 "" H 1700 3000 50  0001 C CNN
+F 3 "" H 1700 3000 50  0001 C CNN
+	1    1700 3000
+	1    0    0    -1
+$EndComp
 Wire Wire Line
 	5000 5700 6450 5700
@@
 Text Label 10800 2050 0    50   ~ 0
 CTS
+Text Label 10800 1750 0    50   ~ 0
+RTS
+Wire Wire Line
+	5450 2800 7400 2800
+Wire Wire Line
+	5650 2850 7750 2850
 Text Label 10800 1950 0    50   ~ 0
-RTS
-Wire Wire Line
-	5450 2800 7400 2800
-Wire Wire Line
-	5650 2850 7750 2850
+F1TX
 Text Label 10800 1850 0    50   ~ 0
-F1TX
-Text Label 10800 1750 0    50   ~ 0
 F1RX
 Wire Wire Line
@@
 Wire Wire Line
 	1950 3650 2450 3650
-Text Label 10800 2250 0    50   ~ 0
-SWDIO
 Text Label 10800 2150 0    50   ~ 0
 SWCLK
@@
 NoConn ~ 3850 8650
 NoConn ~ 5050 8650
+Text Label 10800 2250 0    50   ~ 0
+SWDIO
+Wire Wire Line
+	7100 3050 7100 2750
+Wire Wire Line
+	7100 2750 4450 2750
+Wire Wire Line
+	7100 3050 7750 3050
+NoConn ~ 4450 3250
+NoConn ~ 4450 3350
+Text Label 2150 1550 3    50   ~ 0
+BOOT0
+Text Label 4450 2450 0    50   ~ 0
+BOOT0
+Wire Wire Line
+	750  900  2150 900
+Text Label 1700 2100 3    50   ~ 0
+BattVolt
+Wire Wire Line
+	1700 2700 2150 2700
+Wire Wire Line
+	2150 2700 2150 2350
+Wire Wire Line
+	2150 2350 2450 2350
+Connection ~ 1700 2700
+Wire Wire Line
+	1700 2400 1700 2050
 $EndSCHEMATC

Commit message: Added changes
Connections:
- net labels added: BOOT1
- wire segments 167 -> 166
- no-connect marks 37 -> 36
Other:
- moved on the sheet: R5
Changed lines of the file:
@@
 L Device:R R5
 U 1 1 5D4A832E
-P 2150 1400
-F 0 "R5" H 2220 1446 50  0000 L CNN
-F 1 "10K" H 2220 1355 50  0000 L CNN
-F 2 "Encoder:R_0603_1608Metric_Pad1.05x0.95mm_HandSolder" V 2080 1400 50  0001 C CNN
-F 3 "~" H 2150 1400 50  0001 C CNN
-	1    2150 1400
-	1    0    0    -1
-$EndComp
-Wire Wire Line
-	2150 1250 2150 900
-Wire Wire Line
-	2150 1550 2150 2050
-Wire Wire Line
-	2150 2050 2450 2050
+P 2050 2200
+F 0 "R5" H 2120 2246 50  0000 L CNN
+F 1 "10K" H 2120 2155 50  0000 L CNN
+F 2 "Encoder:R_0603_1608Metric_Pad1.05x0.95mm_HandSolder" V 1980 2200 50  0001 C CNN
+F 3 "~" H 2050 2200 50  0001 C CNN
+	1    2050 2200
+	1    0    0    -1
+$EndComp
 Text Label 2100 3550 0    50   ~ 0
 SWDIO
@@
 	1    0    0    -1
 $EndComp
-Connection ~ 2150 900
-Wire Wire Line
-	2150 900  3200 900
 Wire Wire Line
 	4450 3050 6900 3050
@@
 NoConn ~ 4450 2250
 NoConn ~ 4450 2350
-NoConn ~ 4450 2450
 NoConn ~ 4450 2650
 Wire Wire Line
@@
 NoConn ~ 4450 3250
 NoConn ~ 4450 3350
-Text Label 2150 1550 3    50   ~ 0
+Text Label 2150 2050 0    50   ~ 0
 BOOT0
 Text Label 4450 2450 0    50   ~ 0
-BOOT0
-Wire Wire Line
-	750  900  2150 900
+BOOT1
 Text Label 1700 2100 3    50   ~ 0
 BattVolt
@@
 Wire Wire Line
 	1700 2400 1700 2050
+Wire Wire Line
+	4450 2450 5350 2450
+Wire Wire Line
+	5350 2450 5350 2500
+$Comp
+L power:GND #PWR0102
+U 1 1 5D535B59
+P 5350 2500
+F 0 "#PWR0102" H 5350 2250 50  0001 C CNN
+F 1 "GND" H 5355 2327 50  0000 C CNN
+F 2 "" H 5350 2500 50  0001 C CNN
+F 3 "" H 5350 2500 50  0001 C CNN
+	1    5350 2500
+	1    0    0    -1
+$EndComp
+Wire Wire Line
+	750  900  3200 900
+Wire Wire Line
+	2050 2050 2450 2050
+$Comp
+L power:GND #PWR?
+U 1 1 5D5484B5
+P 2050 2350
+F 0 "#PWR?" H 2050 2100 50  0001 C CNN
+F 1 "GND" H 2055 2177 50  0000 C CNN
+F 2 "" H 2050 2350 50  0001 C CNN
+F 3 "" H 2050 2350 50  0001 C CNN
+	1    2050 2350
+	1    0    0    -1
+$EndComp
 $EndSCHEMATC

Commit message: Added changes
Parts:
- added Q3: Q_PMOS_GSD, Encoder:SOT-23, symbol Encoder:Q_PMOS_GSD
Connections:
- net labels added: EncEnable
- wire segments 166 -> 175
- no-connect marks 36 -> 37
Other:
- moved on the sheet: C2, R1, R13, R14, R2, R3, R4, R5, U2, U3

Commit message: Added changes
Parts:
- added C17: 10uF, Encoder:C_0603_1608Metric_Pad1.05x0.95mm_HandSolder, symbol Device:C
- added D2: D, Encoder:D_SMA, symbol Device:D
Connections:
- net labels added: Batt+, Batt-, GNDPWR
- net labels removed: BattVolt
- wire segments 175 -> 177
Other:
- moved on the sheet: C11, C12, C13, C14, C16, D1, IC2, IC3, J4, J5, J7, Q1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
