File: Mechatronics/Hardware/Electrical/BEncoderBoard/EncoderBoard.sch (KiCad schematic (older format))
At the start: 48 parts, among them IC1 RN4020-V_RM120, IC2 TP4056, IC3 DW01+G, J1 Conn_01x07_Male, J4 Barrel_Jack_Switch, J5 Batt+, J7 Batt-, Q1 FS8205, Q2 Q_PMOS_GSD, Q3 Q_PMOS_GSD, U1 STM32F103C8T6, U2 ITR1802A, U3 ITR1802B, U5 SSD1306OLED, U6 LTC2430, Y1 8Mhz

Commit message: Added changes
Parts:
- removed J4: Barrel_Jack_Switch, Encoder:BarrelJack_Horizontal, symbol Connector:Barrel_Jack_Switch
- added J2: VCC, Encoder:No3dmodelPinHeader_1x01_P2.54mm_Vertical, symbol Connector:Conn_01x01_Male
- added J3, J4: GND, Encoder:No3dmodelPinHeader_1x01_P2.54mm_Vertical, symbol Connector:Conn_01x01_Male
Changed lines of the file:
@@
 Wire Wire Line
 	6000 6750 5700 6750
-$Comp
-L Connector:Barrel_Jack_Switch J4
-U 1 1 5D5D067D
-P 1200 5800
-F 0 "J4" H 1255 6117 50  0000 C CNN
-F 1 "Barrel_Jack_Switch" H 1255 6026 50  0000 C CNN
-F 2 "Encoder:BarrelJack_Horizontal" H 1250 5760 50  0001 C CNN
-F 3 "~" H 1250 5760 50  0001 C CNN
-	1    1200 5800
-	1    0    0    -1
-$EndComp
 Wire Wire Line
 	2050 5900 2050 5800
@@
 Wire Wire Line
 	6200 8050 6600 8050
+$Comp
+L Connector:Conn_01x01_Male J2
+U 1 1 5D5761FD
+P 1300 5700
+F 0 "J2" H 1600 5750 50  0000 R CNN
+F 1 "VCC" H 1273 5721 50  0000 R CNN
+F 2 "Encoder:No3dmodelPinHeader_1x01_P2.54mm_Vertical" H 1300 5700 50  0001 C CNN
+F 3 "~" H 1300 5700 50  0001 C CNN
+	1    1300 5700
+	1    0    0    -1
+$EndComp
+$Comp
+L Connector:Conn_01x01_Male J3
+U 1 1 5D576465
+P 1300 5800
+F 0 "J3" H 1600 5850 50  0000 R CNN
+F 1 "GND" H 1273 5821 50  0000 R CNN
+F 2 "Encoder:No3dmodelPinHeader_1x01_P2.54mm_Vertical" H 1300 5800 50  0001 C CNN
+F 3 "~" H 1300 5800 50  0001 C CNN
+	1    1300 5800
+	1    0    0    -1
+$EndComp
+$Comp
+L Connector:Conn_01x01_Male J4
+U 1 1 5D5766CD
+P 1300 5900
+F 0 "J4" H 1600 5950 50  0000 R CNN
+F 1 "GND" H 1273 5921 50  0000 R CNN
+F 2 "Encoder:No3dmodelPinHeader_1x01_P2.54mm_Vertical" H 1300 5900 50  0001 C CNN
+F 3 "~" H 1300 5900 50  0001 C CNN
+	1    1300 5900
+	1    0    0    -1
+$EndComp
 $EndSCHEMATC

Commit message: Added changes
Parts:
- removed J2: VCC, Encoder:No3dmodelPinHeader_1x01_P2.54mm_Vertical, symbol Connector:Conn_01x01_Male
- removed J3, J4: GND, Encoder:No3dmodelPinHeader_1x01_P2.54mm_Vertical, symbol Connector:Conn_01x01_Male
- added J4: Barrel_Jack_Switch, Encoder:BarrelJack_Horizontal, symbol Connector:Barrel_Jack_Switch
Changed lines of the file:
@@
 	6200 8050 6600 8050
 $Comp
-L Connector:Conn_01x01_Male J2
-U 1 1 5D5761FD
-P 1300 5700
-F 0 "J2" H 1600 5750 50  0000 R CNN
-F 1 "VCC" H 1273 5721 50  0000 R CNN
-F 2 "Encoder:No3dmodelPinHeader_1x01_P2.54mm_Vertical" H 1300 5700 50  0001 C CNN
-F 3 "~" H 1300 5700 50  0001 C CNN
-	1    1300 5700
+L Connector:Barrel_Jack_Switch J4
+U 1 1 5D5D067D
+P 1200 5800
+F 0 "J4" H 1255 6117 50  0000 C CNN
+F 1 "Barrel_Jack_Switch" H 1255 6026 50  0000 C CNN
+F 2 "Encoder:BarrelJack_Horizontal" H 1250 5760 50  0001 C CNN
+F 3 "~" H 1250 5760 50  0001 C CNN
+	1    1200 5800
 	1    0    0    -1
 $EndComp
-$Comp
-L Connector:Conn_01x01_Male J3
-U 1 1 5D576465
-P 1300 5800
-F 0 "J3" H 1600 5850 50  0000 R CNN
-F 1 "GND" H 1273 5821 50  0000 R CNN
-F 2 "Encoder:No3dmodelPinHeader_1x01_P2.54mm_Vertical" H 1300 5800 50  0001 C CNN
-F 3 "~" H 1300 5800 50  0001 C CNN
-	1    1300 5800
-	1    0    0    -1
-$EndComp
-$Comp
-L Connector:Conn_01x01_Male J4
-U 1 1 5D5766CD
-P 1300 5900
-F 0 "J4" H 1600 5950 50  0000 R CNN
-F 1 "GND" H 1273 5921 50  0000 R CNN
-F 2 "Encoder:No3dmodelPinHeader_1x01_P2.54mm_Vertical" H 1300 5900 50  0001 C CNN
-F 3 "~" H 1300 5900 50  0001 C CNN
-	1    1300 5900
-	1    0    0    -1
-$EndComp

Commit message: Added changes
Parts:
- removed D2: D, Encoder:D_SMA, symbol Device:D
- added C18: 1uF, Encoder:C_0603_1608Metric_Pad1.05x0.95mm_HandSolder, symbol Device:C
- added U4: 82402305, Encoder:Sot-23(6), symbol Encoder:82402305
- C17: value 10uF -> 1uF
Connections:
- wire segments 177 -> 176
- no-connect marks 37 -> 43
Other:
- moved on the sheet: C11, C12, C13, C14, C16, D1, IC2, IC3, J5, J7, Q1, Q2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

Commit message: Added changes
Parts:
- removed U6: LTC2430, Encoder:DFN-6_DC, symbol Encoder:LTC2430
- added J2: GNDPWR, Encoder:No3dmodelPinHeader_1x01_P2.54mm_Vertical, symbol Connector:Conn_01x01_Male
- added U6: LTC3240, Encoder:DFN-6_DC, symbol Encoder:LTC3240
Connections:
- wire segments 176 -> 177
Other:
- moved on the sheet: C17, C18, J7, U4
Changed lines of the file:
@@
-$EndComp
-$Comp
-L Encoder:LTC2430 U6
-U 1 1 5D41A14E
-P 10250 6700
-F 0 "U6" H 10275 7265 50  0000 C CNN
-F 1 "LTC2430" H 10275 7174 50  0000 C CNN
-F 2 "Encoder:DFN-6_DC" H 10250 6700 50  0001 C CNN
-F 3 "" H 10250 6700 50  0001 C CNN
-	1    10250 6700
-	1    0    0    -1
 $EndComp
 $Comp
@@
 Wire Wire Line
 	6600 7550 6500 7550
-Wire Wire Line
-	6600 7550 6600 8050
-Connection ~ 6600 7550
-Wire Wire Line
-	6600 8050 6800 8050
-Connection ~ 6600 8050
 $Comp
 L Connector:Conn_01x01_Male J7
 U 1 1 5D5B91B7
-P 7200 7850
-F 0 "J7" H 7173 7780 50  0000 R CNN
-F 1 "Batt-" H 7173 7871 50  0000 R CNN
-F 2 "Encoder:No3dmodelPinHeader_1x01_P2.54mm_Vertical" H 7200 7850 50  0001 C CNN
-F 3 "~" H 7200 7850 50  0001 C CNN
-	1    7200 7850
+P 7650 7850
+F 0 "J7" H 7623 7780 50  0000 R CNN
+F 1 "Batt-" H 7623 7871 50  0000 R CNN
+F 2 "Encoder:No3dmodelPinHeader_1x01_P2.54mm_Vertical" H 7650 7850 50  0001 C CNN
+F 3 "~" H 7650 7850 50  0001 C CNN
+	1    7650 7850
 	0    1    1    0
 $EndComp
@@
 $EndComp
 Wire Wire Line
-	6600 8900 5050 8900
+	7050 8900 5050 8900
 Wire Wire Line
 	5050 8900 5050 8750
@@
 	5050 8750 5150 8750
 Wire Wire Line
-	6600 8050 6600 8900
+	7050 8050 7050 8900
 $Comp
 L Connector:Conn_01x01_Male J5
@@
 Text Label 6850 6750 0    50   ~ 0
 Batt+
-Text Label 6850 8050 0    50   ~ 0
+Text Label 7300 8050 0    50   ~ 0
 Batt-
 Text Label 1600 2350 1    50   ~ 0
 Batt+
 Wire Wire Line
-	3500 7000 3500 7400
-Text Label 3500 7100 3    50   ~ 0
+	2600 7100 2600 7500
+Text Label 2600 7200 3    50   ~ 0
 Batt-
 Wire Wire Line
-	2050 5700 2400 5700
+	2050 5700 2600 5700
 $Comp
 L Device:C C17
 U 1 1 5D58B44B
-P 2400 5850
-F 0 "C17" H 2515 5896 50  0000 L CNN
-F 1 "1uF" H 2515 5805 50  0000 L CNN
-F 2 "Encoder:C_0603_1608Metric_Pad1.05x0.95mm_HandSolder" H 2438 5700 50  0001 C CNN
-F 3 "~" H 2400 5850 50  0001 C CNN
-	1    2400 5850
-	1    0    0    -1
-$EndComp
-Connection ~ 2400 5700
-Wire Wire Line
-	2800 6000 2800 6400
+P 3050 5850
+F 0 "C17" H 3165 5896 50  0000 L CNN
+F 1 "1uF" H 3165 5805 50  0000 L CNN
+F 2 "Encoder:C_0603_1608Metric_Pad1.05x0.95mm_HandSolder" H 3088 5700 50  0001 C CNN
+F 3 "~" H 3050 5850 50  0001 C CNN
+	1    3050 5850
+	1    0    0    -1
+$EndComp
+Connection ~ 3050 5700
+Wire Wire Line
+	3450 6000 3450 6400
 $Comp
 L power:GNDPWR #PWR026
 U 1 1 5D5A0D11
-P 2800 6400
-F 0 "#PWR026" H 2800 6200 50  0001 C CNN
-F 1 "GNDPWR" H 2804 6246 50  0000 C CNN
-F 2 "" H 2800 6350 50  0001 C CNN
-F 3 "" H 2800 6350 50  0001 C CNN
-	1    2800 6400
+P 3450 6400
+F 0 "#PWR026" H 3450 6200 50  0001 C CNN
+F 1 "GNDPWR" H 3454 6246 50  0000 C CNN
+F 2 "" H 3450 6350 50  0001 C CNN
+F 3 "" H 3450 6350 50  0001 C CNN
+	1    3450 6400
 	1    0    0    -1
 $EndComp
@@
 L power:GNDPWR #PWR027
 U 1 1 5D5A0E73
-P 3500 7400
-F 0 "#PWR027" H 3500 7200 50  0001 C CNN
-F 1 "GNDPWR" H 3504 7246 50  0000 C CNN
-F 2 "" H 3500 7350 50  0001 C CNN
-F 3 "" H 3500 7350 50  0001 C CNN
-	1    3500 7400
+P 2600 7500
+F 0 "#PWR027" H 2600 7300 50  0001 C CNN
+F 1 "GNDPWR" H 2604 7346 50  0000 C CNN
+F 2 "" H 2600 7450 50  0001 C CNN
+F 3 "" H 2600 7450 50  0001 C CNN
+	1    2600 7500
 	1    0    0    -1
 $EndComp
@@
 L power:GNDPWR #PWR039
 U 1 1 5D5A1C8E
-P 6800 8050
-F 0 "#PWR039" H 6800 7850 50  0001 C CNN
-F 1 "GNDPWR" H 6804 7896 50  0000 C CNN
-F 2 "" H 6800 8000 50  0001 C CNN
-F 3 "" H 6800 8000 50  0001 C CNN
-	1    6800 8050
-	1    0    0    -1
-$EndComp
-Connection ~ 6800 8050
-Wire Wire Line
-	6800 8050 7200 8050
+P 6550 8650
+F 0 "#PWR039" H 6550 8450 50  0001 C CNN
+F 1 "GNDPWR" H 6554 8496 50  0000 C CNN
+F 2 "" H 6550 8600 50  0001 C CNN
+F 3 "" H 6550 8600 50  0001 C CNN
+	1    6550 8650
+	1    0    0    -1
+$EndComp
 $Comp
 L Connector:Barrel_Jack_Switch J4
@@
 L Encoder:82402305 U4
 U 1 1 5D5CA4C0
-P 3500 6650
-F 0 "U4" H 3778 6696 50  0000 L CNN
-F 1 "82402305" H 3778 6605 50  0000 L CNN
-F 2 "Encoder:Sot-23(6)" H 3500 6600 50  0001 C CNN
-F 3 "" H 3500 6600 50  0001 C CNN
-	1    3500 6650
-	1    0    0    -1
-$EndComp
-Wire Wire Line
-	3500 6300 3500 5700
-Wire Wire Line
-	2400 5700 2800 5700
-Connection ~ 3500 5700
-Wire Wire Line
-	3500 5700 3850 5700
-NoConn ~ 3300 6300
-NoConn ~ 3650 6300
-NoConn ~ 3300 7000
-NoConn ~ 3650 7000
+P 2600 6750
+F 0 "U4" H 2878 6796 50  0000 L CNN
+F 1 "82402305" H 2878 6705 50  0000 L CNN
+F 2 "Encoder:Sot-23(6)" H 2600 6700 50  0001 C CNN
+F 3 "" H 2600 6700 50  0001 C CNN
+	1    2600 6750
+	1    0    0    -1
+$EndComp
+Wire Wire Line
+	3050 5700 3450 5700
+NoConn ~ 2400 6400
+NoConn ~ 2750 6400
+NoConn ~ 2400 7100
+NoConn ~ 2750 7100
 $Comp
 L Device:C C18
 U 1 1 5D631F29
-P 2800 5850
-F 0 "C18" H 2915 5896 50  0000 L CNN
-F 1 "1uF" H 2915 5805 50  0000 L CNN
-F 2 "Encoder:C_0603_1608Metric_Pad1.05x0.95mm_HandSolder" H 2838 5700 50  0001 C CNN
-F 3 "~" H 2800 5850 50  0001 C CNN
-	1    2800 5850
-	1    0    0    -1
-$EndComp
-Connection ~ 2800 5700
-Wire Wire Line
-	2800 5700 3500 5700
-Wire Wire Line
-	2400 6000 2400 6400
+P 3450 5850
+F 0 "C18" H 3565 5896 50  0000 L CNN
+F 1 "1uF" H 3565 5805 50  0000 L CNN
+F 2 "Encoder:C_0603_1608Metric_Pad1.05x0.95mm_HandSolder" H 3488 5700 50  0001 C CNN
+F 3 "~" H 3450 5850 50  0001 C CNN
+	1    3450 5850
+	1    0    0    -1
+$EndComp
+Connection ~ 3450 5700
+Wire Wire Line
+	3050 6000 3050 6400
 $Comp
 L power:GNDPWR #PWR040
 U 1 1 5D63C3AA
-P 2400 6400
-F 0 "#PWR040" H 2400 6200 50  0001 C CNN
-F 1 "GNDPWR" H 2404 6246 50  0000 C CNN
-F 2 "" H 2400 6350 50  0001 C CNN
-F 3 "" H 2400 6350 50  0001 C CNN
-	1    2400 6400
+P 3050 6400
+F 0 "#PWR040" H 3050 6200 50  0001 C CNN
+F 1 "GNDPWR" H 3054 6246 50  0000 C CNN
+F 2 "" H 3050 6350 50  0001 C CNN
+F 3 "" H 3050 6350 50  0001 C CNN
+	1    3050 6400
 	1    0    0    -1
 $EndComp
 NoConn ~ 5150 8550
 $Comp
-L power:GND #PWR?
+L power:GND #PWR0103
 U 1 1 5D665A31
-P 6500 8650
-F 0 "#PWR?" H 6500 8400 50  0001 C CNN
-F 1 "GND" H 6505 8477 50  0000 C CNN
-F 2 "" H 6500 8650 50  0001 C CNN
-F 3 "" H 6500 8650 50  0001 C CNN
-	1    6500 8650
+P 6850 8650
+F 0 "#PWR0103" H 6850 8400 50  0001 C CNN
+F 1 "GND" H 6855 8477 50  0000 C CNN
+F 2 "" H 6850 8650 50  0001 C CNN
+F 3 "" H 6850 8650 50  0001 C CNN
+	1    6850 8650
 	-1   0    0    -1
 $EndComp
-Wire Wire Line
-	6500 8650 6350 8650
 NoConn ~ 5150 8650
 NoConn ~ 6350 8750
 NoConn ~ 5500 7750
+Wire Wire Line
+	7050 8050 7650 8050
+Wire Wire Line
+	6600 7550 6600 8050
+Wire Wire Line
+	6600 8050 7050 8050
+Connection ~ 6600 7550
+Connection ~ 7050 8050
+Wire Wire Line
+	6350 8650 6550 8650
+Connection ~ 6550 8650
+Wire Wire Line
+	6550 8650 6850 8650
+$Comp
+L Connector:Conn_01x01_Male J2
+U 1 1 5D611BB9
+P 1900 7500
+F 0 "J2" H 1873 7430 50  0000 R CNN
+F 1 "GNDPWR" H 1873 7521 50  0000 R CNN
+F 2 "Encoder:No3dmodelPinHeader_1x01_P2.54mm_Vertical" H 1900 7500 50  0001 C CNN
+F 3 "~" H 1900 7500 50  0001 C CNN
+	1    1900 7500
+	0    1    1    0
+$EndComp
+$Comp
+L power:GNDPWR #PWR036
+U 1 1 5D611C3F
+P 1900 7700
+F 0 "#PWR036" H 1900 7500 50  0001 C CNN
+F 1 "GNDPWR" H 1904 7546 50  0000 C CNN
+F 2 "" H 1900 7650 50  0001 C CNN
+F 3 "" H 1900 7650 50  0001 C CNN
+	1    1900 7700
+	1    0    0    -1
+$EndComp
+$Comp
+L Encoder:LTC3240 U6
+U 1 1 5D5E0FAC
+P 10250 6700
+F 0 "U6" H 10275 7265 50  0000 C CNN
+F 1 "LTC3240" H 10275 7174 50  0000 C CNN
+F 2 "Encoder:DFN-6_DC" H 10250 6700 50  0001 C CNN
+F 3 "" H 10250 6700 50  0001 C CNN
+	1    10250 6700
+	1    0    0    -1
+$EndComp
+Wire Wire Line
+	3450 5700 3850 5700
+Wire Wire Line
+	2600 6400 2600 5700
+Connection ~ 2600 5700
+Wire Wire Line
+	2600 5700 3050 5700
 $EndSCHEMATC

Commit message: Added changes
Connections:
- net labels removed: STDBY
- wire segments 177 -> 179
- no-connect marks 43 -> 44

Commit message: Added changes
Parts:
- U2: value ITR1802A -> ITR1802
- U3: value ITR1802B -> ITR1802
Changed lines of the file:
@@
 P 14550 2400
 F 0 "U2" H 14550 2725 50  0000 C CNN
-F 1 "ITR1802A" H 14550 2634 50  0000 C CNN
+F 1 "ITR1802" H 14550 2634 50  0000 C CNN
 F 2 "Encoder:OptointerrupterConnector" H 14550 2400 50  0001 C CNN
 F 3 "" H 14550 2400 50  0001 C CNN
@@
 P 14550 2950
 F 0 "U3" H 14550 3275 50  0000 C CNN
-F 1 "ITR1802B" H 14550 3184 50  0000 C CNN
+F 1 "ITR1802" H 14550 3184 50  0000 C CNN
 F 2 "Encoder:OptointerrupterConnector" H 14550 2950 50  0001 C CNN
 F 3 "" H 14550 2950 50  0001 C CNN

Commit message: Added changes
Other:
- moved on the sheet: Q3
Changed lines of the file:
@@
 L Encoder:Q_PMOS_GSD Q3
 U 1 1 5D553268
-P 14400 1550
-F 0 "Q3" H 14500 1350 50  0000 C CNN
-F 1 "Q_PMOS_GSD" H 14500 1250 50  0000 C CNN
-F 2 "Encoder:SOT-23" V 14600 1400 50  0001 C CNN
-F 3 "~" V 14400 1600 50  0001 C CNN
-	1    14400 1550
+P 14400 1600
+F 0 "Q3" H 14500 1400 50  0000 C CNN
+F 1 "Q_PMOS_GSD" H 14500 1300 50  0000 C CNN
+F 2 "Encoder:SOT-23" V 14600 1450 50  0001 C CNN
+F 3 "~" V 14400 1650 50  0001 C CNN
+	1    14400 1600
 	1    0    0    -1
 $EndComp
@@
 Text Label 2100 2650 0    50   ~ 0
 EncEnable
-Text Label 14400 1150 1    50   ~ 0
+Text Label 14400 1200 1    50   ~ 0
 EncEnable
 Wire Wire Line
-	14400 1300 14400 750
+	14400 1350 14400 800
 Wire Wire Line
-	14200 1600 14200 1950
+	14200 1650 14200 2000
 $Comp
 L power:+3.3V #PWR017
 U 1 1 5D59FF5B
-P 14600 1600
-F 0 "#PWR017" H 14600 1450 50  0001 C CNN
-F 1 "+3.3V" H 14615 1773 50  0000 C CNN
-F 2 "" H 14600 1600 50  0001 C CNN
-F 3 "" H 14600 1600 50  0001 C CNN
-	1    14600 1600
+P 14600 1650
+F 0 "#PWR017" H 14600 1500 50  0001 C CNN
+F 1 "+3.3V" H 14615 1823 50  0000 C CNN
+F 2 "" H 14600 1650 50  0001 C CNN
+F 3 "" H 14600 1650 50  0001 C CNN
+	1    14600 1650
 	1    0    0    -1
 $EndComp
 Wire Wire Line
-	15100 2200 15100 1950
+	15100 2200 15100 2000
 Wire Wire Line
-	15100 1950 14200 1950
-Connection ~ 14200 1950
+	15100 2000 14200 2000
+Connection ~ 14200 2000
 Wire Wire Line
-	14200 1950 14200 2300
+	14200 2000 14200 2300
 Wire Wire Line
 	15100 2750 15750 2750
 Wire Wire Line
-	15750 2750 15750 1950
+	15750 2750 15750 2000
 Wire Wire Line
-	15750 1950 15100 1950
-Connection ~ 15100 1950
+	15750 2000 15100 2000
+Connection ~ 15100 2000
 Wire Wire Line
 	6600 6750 7150 6750
