File: Mechatronics/Hardware/Electrical/BEncoderBoard/EncoderBoard.sch (KiCad schematic (older format))
At the start: 50 parts, among them IC1 RN4020-V_RM120, IC2 TP4056, IC3 DW01+G, J1 Conn_01x07_Male, J2 GNDPWR, J4 Barrel_Jack_Switch, J5 Batt+, J7 Batt-, Q1 FS8205, Q2 Q_PMOS_GSD, Q3 Q_PMOS_GSD, U1 STM32F103C8T6, U2 ITR1802, U3 ITR1802, U5 SSD1306OLED, U6 LTC3240, Y1 8Mhz

Commit message: Added changes
Parts:
- removed D2: D, Diode_THT:D_DO-201AD_P5.08mm_Vertical_AnodeUp, symbol Device:D
- removed Q1: FS8205, Encoder:Sot-23(6), symbol Encoder:FS8205
- added Q1: DMosfet, Encoder:Sot-23(6), symbol Encoder:DMosfet
- added U4: 82402305, Encoder:Sot-23(6), symbol Encoder:82402305
- U1: Campo4 Unavailable -> (none); Campo5 None -> (none); Campo6 Mainstream Performance line, ARM Cortex-M3 MCU with 64 Kbyt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 -> (none); Campo7 STMicroelectronics -> (none); Campo8 LQFP-48 STMicroelectronics -> (none); Field4 (none) -> Unavailable; Field5 (none) -> None; Field6 (none) -> Mainstream Performance line, ARM Cortex-M3 MCU with 64 Kbyt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; Field7 (none) -> STMicroelectronics; Field8 (none) -> LQFP-48 STMicroelectronics
Connections:
- wire segments 179 -> 178
Other:
- moved on the sheet: C11, C12, C13, C14, C15, C16, C17, C18, D1, IC1, IC2, IC3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

Commit message: Added changes
Connections:
- wire segments 178 -> 177
Changed lines of the file:
@@
 Batt-
 Wire Wire Line
-	2800 7150 2800 7350
-Wire Wire Line
 	2800 7350 2800 7550
-Connection ~ 2800 7350
 Wire Wire Line
 	8950 6700 9150 6700

Commit message: Added changes
Connections:
- net labels added: RN4020RX, RN4020TX
Changed lines of the file:
@@
 NoConn ~ 9950 3350
-$Comp
-L power:GND #PWR030
-U 1 1 5D4A2EDD
-P 9950 2750
-F 0 "#PWR030" H 9950 2500 50  0001 C CNN
-F 1 "GND" H 9955 2577 50  0000 C CNN
-F 2 "" H 9950 2750 50  0001 C CNN
-F 3 "" H 9950 2750 50  0001 C CNN
-	1    9950 2750
-	0    -1   -1   0
-$EndComp
-$Comp
-L power:GND #PWR029
-U 1 1 5D4A2F83
-P 8050 3250
-F 0 "#PWR029" H 8050 3000 50  0001 C CNN
-F 1 "GND" H 8055 3077 50  0000 C CNN
-F 2 "" H 8050 3250 50  0001 C CNN
-F 3 "" H 8050 3250 50  0001 C CNN
-	1    8050 3250
-	0    1    1    0
-$EndComp
 $Comp
 L power:GND #PWR028
@@
 Wire Wire Line
 	5650 2850 8050 2850
-Text Label 11200 1550 0    50   ~ 0
-F1TX
-Text Label 11200 1450 0    50   ~ 0
-F1RX
+Text Label 11050 1550 0    50   ~ 0
+RN4020RX
 Wire Wire Line
 	1950 3550 2450 3550
@@
 	9300 6900 9150 6900
 Connection ~ 9300 6900
+Text Label 11050 1450 0    50   ~ 0
+RN4020TX
+Text Label 7550 2850 0    50   ~ 0
+RN4020TX
+Text Label 7550 2950 0    50   ~ 0
+RN4020RX
 $EndSCHEMATC

Commit message: Added changes
Parts:
- added R10, R12, R15, R16: 10K, Encoder:R_0603_1608Metric_Pad1.05x0.95mm_HandSolder, symbol Device:R
Connections:
- wire segments 177 -> 180
Other:
- moved on the sheet: J1, Q3, R1, R2, R3, R4, U2, U3

Commit message: New Changes
Parts:
- IC2: symbol Encoder:TP4056 -> EncoderBoard-rescue:TP4056-Encoder
- IC3: symbol Encoder:DW01+G -> EncoderBoard-rescue:DW01+G-Encoder
- J1: footprint Encoder:PinSocket_1x07_P2.54mm_Vertical -> Encoder:PinHeader_1x07_P2.54mm_Vertical
- J5, J7: footprint Encoder:No3dmodelPinHeader_1x01_P2.54mm_Vertical -> Encoder:PinHeader_1x01_P2.54mm_Vertical_NO3D
- U1: footprint Encoder:QFP50P900X900X160-48N -> Encoder:LQFP-48_7x7mm_P0.5mm
- U4: symbol Encoder:82402305 -> EncoderBoard-rescue:82402305-Encoder
Changed lines of the file:
@@
 EESchema Schematic File Version 4
-LIBS:EncoderBoard-cache
 EELAYER 30 0
 EELAYER END
@@
 Connection ~ 6500 5750
 $Comp
-L Encoder:DW01+G IC3
+L EncoderBoard-rescue:DW01+G-Encoder IC3
 U 1 1 5D56FBF8
 P 5700 7600
@@
 F 0 "J7" H 7823 7830 50  0000 R CNN
 F 1 "Batt-" H 7823 7921 50  0000 R CNN
-F 2 "Encoder:No3dmodelPinHeader_1x01_P2.54mm_Vertical" H 7850 7900 50  0001 C CNN
+F 2 "Encoder:PinHeader_1x01_P2.54mm_Vertical_NO3D" H 7850 7900 50  0001 C CNN
 F 3 "~" H 7850 7900 50  0001 C CNN
 	1    7850 7900
@@
 F 0 "J5" H 7323 6530 50  0000 R CNN
 F 1 "Batt+" H 7323 6621 50  0000 R CNN
-F 2 "Encoder:No3dmodelPinHeader_1x01_P2.54mm_Vertical" H 7350 6600 50  0001 C CNN
+F 2 "Encoder:PinHeader_1x01_P2.54mm_Vertical_NO3D" H 7350 6600 50  0001 C CNN
 F 3 "~" H 7350 6600 50  0001 C CNN
 	1    7350 6600
@@
 	4400 6800 5100 6800
 $Comp
-L Encoder:TP4056 IC2
+L EncoderBoard-rescue:TP4056-Encoder IC2
 U 1 1 5D4C3075
 P 5100 6500
@@
 F 0 "J1" H 9573 1280 50  0000 R CNN
 F 1 "Conn_01x07_Male" H 9573 1371 50  0000 R CNN
-F 2 "Encoder:PinSocket_1x07_P2.54mm_Vertical" H 9600 1350 50  0001 C CNN
+F 2 "Encoder:PinHeader_1x07_P2.54mm_Vertical" H 9600 1350 50  0001 C CNN
 F 3 "~" H 9600 1350 50  0001 C CNN
 	1    9600 1350
@@
 F 0 "U1" H 3450 4817 50  0000 C CNN
 F 1 "STM32F103C8T6" H 3450 4726 50  0000 C CNN
-F 2 "Encoder:QFP50P900X900X160-48N" H 3450 3050 50  0001 L BNN
+F 2 "Encoder:LQFP-48_7x7mm_P0.5mm" H 3450 3050 50  0001 L BNN
 F 3 "STM32F103C8T6" H 3450 3050 50  0001 L BNN
 F 4 "Unavailable" H 3450 3050 50  0001 L BNN "Field4"
@@
 $EndComp
 $Comp
-L Encoder:82402305 U4
+L EncoderBoard-rescue:82402305-Encoder U4
 U 1 1 5D8F0F67
 P 2800 6800
