File: Mechatronics/Hardware/Electrical/BEncoderBoard/EncoderBoard.kicad_pcb (KiCad board)
At the start: 2 copper layers, 66 x 77.5 mm, 32 parts, among them J1 Conn_01x01_Male, J10 Conn_01x01_Male, J2 Conn_01x01_Male, J3 Conn_01x01_Male, J4 Conn_01x01_Male, J5 Conn_01x01_Male, J6 Conn_01x01_Male, J7 Conn_01x01_Male, J8 Conn_01x01_Male, J9 Conn_01x01_Male, Q1 Q_NMOS_SGD, Q2 Q_NMOS_SGD, Q3 Q_NMOS_SGD, U1 ATmega328-PU, U2 ITR1802A, U3 ITR1802B, U4 HEF40106BT, Y1 20Mhz

Commit message: Changes
Parts:
- removed Q2, Q3: Q_NMOS_SGD, Encoder:TO-92_Inline_Wide
- removed R10, R8, R9: 10K, Encoder:R_Axial_DIN0414_L11.9mm_D4.5mm_P15.24mm_Horizontal
- added C10: 100nF, Encoder:C_0603_1608Metric_Pad1.05x0.95mm_HandSolder, F.Cu at (122.9, 116.3)
- added C11: 1uF, Encoder:C_0603_1608Metric_Pad1.05x0.95mm_HandSolder, F.Cu at (201.9, 122.4)
- added C12: 4.7uF, Encoder:C_0603_1608Metric_Pad1.05x0.95mm_HandSolder, F.Cu at (253.2, 104.1)
- added C14: 1uF, Encoder:C_0603_1608Metric_Pad1.05x0.95mm_HandSolder, F.Cu at (213.1, 125.0)
- added C15: 4.7uF, Encoder:C_0603_1608Metric_Pad1.05x0.95mm_HandSolder, F.Cu at (128.0, 93.5)
- added C5: 100nF, Encoder:C_0603_1608Metric_Pad1.05x0.95mm_HandSolder, F.Cu at (123.6, 107.9)
- added C6: 10uF, Encoder:C_0603_1608Metric_Pad1.05x0.95mm_HandSolder, F.Cu at (133.9, 107.7)
- added C7: 12pF, Encoder:C_0603_1608Metric_Pad1.05x0.95mm_HandSolder, F.Cu at (100.7, 108.5)
- added C8: 12pF, Encoder:C_0603_1608Metric_Pad1.05x0.95mm_HandSolder, F.Cu at (100.7, 111.6)
- added C9: 100nF, Encoder:C_0603_1608Metric_Pad1.05x0.95mm_HandSolder, F.Cu at (113.4, 106.2)
- added D1: TVS, Encoder:D_DO-201AD_P15.24mm_Horizontal, F.Cu at (199.1, 105.8)
- added D2: D_Schottky, Encoder:D_DO-201AD_P15.24mm_Horizontal, F.Cu at (180.1, 101.9)
- added IC1: RN4020-V_RM120, Encoder:Bluetooth_Module_RN4020, F.Cu at (119.5, 98.1)
- added J12: Batt-, Encoder:PinHeader_1x01_P2.54mm_Vertical, F.Cu at (230.2, 104.5)
- added S1: EG1218, Encoder:Switch_Slide_11.6x4mm_EG1218, F.Cu at (181.9, 107.1)
- added U5: SSD1306OLED, Encoder:SSD1306, F.Cu at (109.0, 98.2)
- added U6: LTC2430, Encoder:DFN-6_DC, F.Cu at (195.4, 106.0)
- C1, C2: value .1uF -> 100nF; footprint Encoder:C_Disc_D9.0mm_W5.0mm_P5.00mm -> Encoder:C_0603_1608Metric_Pad1.05x0.95mm_HandSolder
- C3: value 22pF -> 100nF; footprint Encoder:C_Disc_D9.0mm_W5.0mm_P5.00mm -> Encoder:C_0603_1608Metric_Pad1.05x0.95mm_HandSolder
- C4: value 22pF -> 1uF; footprint Encoder:C_Disc_D9.0mm_W5.0mm_P5.00mm -> Encoder:C_0603_1608Metric_Pad1.05x0.95mm_HandSolder
- J10: value Conn_01x01_Male -> F1RX
- J8: value Conn_01x01_Male -> Batt+
- J9: value Conn_01x01_Male -> F1TX
- Q1: value Q_NMOS_SGD -> Q_PMOS_GDS; footprint Encoder:TO-92_Inline_Wide -> Encoder:TO-220-3_Horizontal_TabDown
- R1, R2, R3, R4, R5, R6, R7: footprint Encoder:R_Axial_DIN0414_L11.9mm_D4.5mm_P15.24mm_Horizontal -> Encoder:R_0603_1608Metric_Pad1.05x0.95mm_HandSolder
- U1: value ATmega328-PU -> STM32F103C8T6; footprint Encoder:DIP-28_W7.62mm_LongPads -> Encoder:QFP50P900X900X160-48N
- U4: value HEF40106BT -> 03962A; footprint Encoder:SOIC-14 -> Encoder:03962A
- Y1: value 20Mhz -> 8Mhz
- moved R6 148.6 mm to (247.2, 96.6), turned to 0 degrees
- moved J7 120.4 mm to (232.3, 91.0), turned to 0 degrees
- moved J4 118.9 mm to (232.3, 87.4)
- moved J8 97.7 mm to (212.6, 110.5), turned to 0 degrees
- moved R7 95.3 mm to (207.0, 122.4), turned to 0 degrees
- moved Q1 93.7 mm to (209.1, 101.6)
- moved J5 86.0 mm to (212.6, 115.0)
- moved U4 77.4 mm to (184.2, 40.6), turned to 0 degrees
- moved R1 50.9 mm to (111.3, 126.2), turned to 0 degrees
- moved U2 48.5 mm to (113.9, 121.6), turned to 0 degrees
- moved J6 45.3 mm to (128.0, 103.4)
- moved U3 44.4 mm to (125.1, 121.7), turned to 0 degrees
- moved R3 43.7 mm to (116.9, 126.2)
- moved R4 43.5 mm to (128.6, 126.2)
- moved J2 40.8 mm to (128.0, 106.9)
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Connections:
- C1 pad 1: GND -> +3V3
- C1 pad 2: +5V -> GND
- C2 pad 1: +5V -> Net-(C2-Pad1)
- C3 pad 2: Net-(C3-Pad2) -> +3V3
- C4 pad 2: Net-(C4-Pad2) -> +3V3
- J1 pad 1: +5V -> /SWCLK
- J10 pad 1: /BattVoltSens -> /F1RX
- J2 pad 1: GND -> Net-(IC1-Pad14)
- J3 pad 1: /3VCMD -> /SWDIO
- J4 pad 1: /3VTX -> VCC
- J5 pad 1: /3VRX -> /Batt+
- J6 pad 1: +3V3 -> Net-(IC1-Pad18)
- J7 pad 1: /SDA -> /Batt-
- J8 pad 1: /SCL -> /Batt+
- J9 pad 1: /PowSupStat -> /F1TX
- Q1 pad 1: /3VCMD -> VCC
- Q1 pad 2: +3V3 -> Net-(D2-Pad1)
- Q1 pad 3: /CMD -> Net-(Q1-Pad3)
- R3 pad 1: +5V -> +3V3
- R4 pad 1: +5V -> +3V3
- R5 pad 2: /3VCMD -> Net-(R5-Pad2)
- R6 pad 1: +3V3 -> VCC
- R6 pad 2: /3VTX -> GND
- R7 pad 1: +3V3 -> Net-(C11-Pad2)
- R7 pad 2: /3VRX -> Net-(R7-Pad2)
- U1 pad 1: (no net) -> +3V3
- U1 pad 10: Net-(C4-Pad2) -> (no net)
- U1 pad 11: (no net) -> /Batt+
- U1 pad 15: /PowSupStat -> (no net)
- U1 pad 2: /RX -> (no net)
- U1 pad 20: +5V -> (no net)
- U1 pad 22: GND -> Net-(IC1-Pad7)
- U1 pad 23: /BattVoltSens -> GND
- U1 pad 24: (no net) -> +3V3
- U1 pad 25: (no net) -> VCC
- U1 pad 27: /SDA -> (no net)
- U1 pad 28: /SCL -> (no net)
- U1 pad 3: /TX -> (no net)
- U1 pad 4: /OUTA -> (no net)
- U1 pad 5: /OUTB -> Net-(C7-Pad2)
- U1 pad 6: /CMD -> Net-(C8-Pad2)
- U1 pad 7: +5V -> Net-(C2-Pad1)
- U1 pad 9: Net-(C3-Pad2) -> +3V3
- U2 pad 1: +5V -> +3V3
- U3 pad 1: +5V -> +3V3
- U4 pad 1: /SIGB -> VCC
- U4 pad 2: /OUTB -> GND
- U4 pad 5: /SIGA -> Net-(Q1-Pad3)
- U4 pad 6: /OUTA -> GND
- Y1 pad 1: Net-(C3-Pad2) -> Net-(C7-Pad2)
- Y1 pad 2: Net-(C4-Pad2) -> Net-(C8-Pad2)
Routing:
- net +5V: track 293.9 -> 0.00 mm
- net +3V3: track 127.7 -> 0.00 mm
- net /SDA: track 77.3 -> 0.00 mm
- net /SCL: track 77.3 -> 0.00 mm
- net /CMD: track 67.3 -> 0.00 mm
- net /TX: track 57.3 -> 0.00 mm
- net /RX: track 45.8 -> 0.00 mm
- net /OUTB: track 41.8 -> 0.00 mm
- net /PowSupStat: track 41.0 -> 0.00 mm
- net /OUTA: track 39.5 -> 0.00 mm
- net /3VTX: track 37.2 -> 0.00 mm
- net /3VRX: track 30.4 -> 0.00 mm
- net Net-(R2-Pad1): track 27.9 -> 3.27 mm
- net /3VCMD: track 21.8 -> 0.00 mm
- net /BattVoltSens: track 19.3 -> 0.00 mm
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- removed copper zone on B.Cu, net GND
Other:
- net class Default: clearance 0.254 -> 0.1016; trace_width 0.254 -> 0.1016
- rule trace_clearance: 0.254 -> 0.1016
- rule trace_min: 0.254 -> 0.0889
- board text removed: "3.3V"
- board text removed: "5V"
- board text removed: "A"
- board text removed: "B"
- board text removed: "BATTS"
- board text removed: "CMD"
- board text removed: "GND"
- board text removed: "PSTAT"
- board text removed: "RX"
- board text removed: "SCL"
- board text removed: "SDA"
- board text removed: "TX"

Commit message: Added changes
Parts:
- removed D2: D_Schottky, Encoder:D_DO-201AD_P15.24mm_Horizontal
- removed J10: F1RX, Encoder:PinHeader_1x01_P2.54mm_Vertical
- removed J12: Batt-, Encoder:PinHeader_1x01_P2.54mm_Vertical
- removed J2, J3, J6: Conn_01x01_Male, Encoder:PinHeader_1x01_P2.54mm_Vertical
- removed J8: Batt+, Encoder:PinHeader_1x01_P2.54mm_Vertical
- removed J9: F1TX, Encoder:PinHeader_1x01_P2.54mm_Vertical
- removed U4: 03962A, Encoder:03962A
- added C13: 10uF, Encoder:C_0603_1608Metric_Pad1.05x0.95mm_HandSolder, F.Cu at (113.1, 144.2)
- added C16: .1uF, Encoder:C_0603_1608Metric_Pad1.05x0.95mm_HandSolder, F.Cu at (120.1, 133.9)
- added IC2: TP4056, Encoder:Sop(8), F.Cu at (115.6, 137.2)
- added IC3: DW01+G, Encoder:Sot-23(6), F.Cu at (121.1, 138.1)
- added Q2: Q_PMOS_GSD, Encoder:SOT-23, F.Cu at (112.6, 127.7)
- added R11: 100, Encoder:R_0603_1608Metric_Pad1.05x0.95mm_HandSolder, F.Cu at (116.1, 128.6)
- added R13: 10K, Encoder:R_0603_1608Metric_Pad1.05x0.95mm_HandSolder, F.Cu at (169.5, 93.9)
- added R14: 10K, Encoder:R_0603_1608Metric_Pad1.05x0.95mm_HandSolder, F.Cu at (169.7, 97.8)
- added R8: 1.2K, Encoder:R_0603_1608Metric_Pad1.05x0.95mm_HandSolder, F.Cu at (114.9, 142.6)
- added R9: 1K, Encoder:R_0603_1608Metric_Pad1.05x0.95mm_HandSolder, F.Cu at (122.0, 141.2)
- D1: value TVS -> D; footprint Encoder:D_DO-201AD_P15.24mm_Horizontal -> Encoder:D_SMA
- J1: value Conn_01x01_Male -> Conn_01x07_Male; footprint Encoder:PinHeader_1x01_P2.54mm_Vertical -> Encoder:PinSocket_1x07_P2.54mm_Vertical
- J4: value Conn_01x01_Male -> Barrel_Jack_Switch; footprint Encoder:PinHeader_1x01_P2.54mm_Vertical -> Encoder:BarrelJack_Horizontal
- J5: value Conn_01x01_Male -> Batt+; footprint Encoder:PinHeader_1x01_P2.54mm_Vertical -> Encoder:No3dmodelPinHeader_1x01_P2.54mm_Vertical
- J7: value Conn_01x01_Male -> Batt-; footprint Encoder:PinHeader_1x01_P2.54mm_Vertical -> Encoder:No3dmodelPinHeader_1x01_P2.54mm_Vertical
- Q1: value Q_PMOS_GDS -> FS8205; footprint Encoder:TO-220-3_Horizontal_TabDown -> Encoder:Sot-23(6)
- U5: footprint Encoder:SSD1306 -> Encoder:PinSocket_1x04_P2.54mm_Vertical
- moved R6 140.6 mm to (110.1, 127.7), turned to 90 degrees
- moved C12 129.7 mm to (126.2, 130.2)
- moved J7 122.8 mm to (116.2, 131.2), turned to 90 degrees
- moved J4 112.0 mm to (132.8, 138.9), turned to 90 degrees
- moved J5 101.3 mm to (112.6, 131.2), turned to 90 degrees
- moved Q1 91.8 mm to (124.8, 138.1), turned to 90 degrees
- moved C14 88.2 mm to (124.9, 125.5)
- moved D1 86.8 mm to (114.3, 124.2), turned to 180 degrees
- moved R7 85.3 mm to (121.8, 126.7), turned to 90 degrees
- moved C11 79.5 mm to (122.8, 130.2)
- moved U6 74.7 mm to (124.0, 127.9), turned to 90 degrees
- moved S1 66.5 mm to (119.4, 129.6), turned to 90 degrees
- moved J1 24.4 mm to (140.9, 89.8)
- moved C10 22.5 mm to (129.5, 94.9)
- moved C15 22.5 mm to (134.6, 72.0)
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Connections:
- net /Batt+ renamed /BattVolt
- D1 pad 1: VCC -> Net-(D1-Pad1)
- D1 pad 2: GND -> VCC
- IC1 pad 14: Net-(IC1-Pad14) -> /CTS
- IC1 pad 18: Net-(IC1-Pad18) -> /RTS
- J1 pad 1: /SWCLK -> /SWDIO
- J7 pad 1: /Batt- -> Net-(C16-Pad2)
- Q1 pad 1: VCC -> GND
- Q1 pad 2: Net-(D2-Pad1) -> (no net)
- Q1 pad 3: Net-(Q1-Pad3) -> Net-(C16-Pad2)
- S1 pad 1: Net-(D2-Pad1) -> Net-(D1-Pad1)
- U1 pad 25: VCC -> /CHG
- U1 pad 26: (no net) -> /STDBY
- U6 pad 7: (no net) -> GND
Routing:
- net VCC: track 0.00 -> 59.3 mm
- net /BattVolt: track 0.00 -> 15.6 mm
- net Net-(IC3-Pad1): track 0.00 -> 15.3 mm
- net Net-(C16-Pad2): track 0.00 -> 15.1 mm
- net Net-(D1-Pad1): track 0.00 -> 12.8 mm
- net Net-(C11-Pad2): track 0.00 -> 11.2 mm
- net Net-(IC3-Pad3): track 0.00 -> 10.8 mm
- net Net-(C16-Pad1): track 0.00 -> 9.98 mm
- net /SIGA: track 28.7 -> 25.0 mm
- net Net-(R7-Pad2): track 0.00 -> 2.22 mm
- net +3V3: track 0.00 -> 2.09 mm
- net Net-(C14-Pad2): track 0.00 -> 2.05 mm
- net Net-(IC3-Pad2): track 0.00 -> 1.86 mm
- net Net-(IC2-Pad2): track 0.00 -> 1.85 mm
- net Net-(C14-Pad1): track 0.00 -> 1.53 mm
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
Commit message: Added changes
Parts:
- J4: moved to B.Cu
- moved J4 0.97 mm to (133.8, 139.3)
Routing:
- net VCC: track 59.3 -> 60.9 mm
Changed lines of the file:
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@@
     (thickness 1.6)
     (drawings 14)
-    (tracks 209)
+    (tracks 213)
     (zones 0)
     (modules 45)
@@
     )
   )
-  (module Encoder:BarrelJack_Horizontal (layer F.Cu)
-    (at 132.842 138.94816 90)
+  (module Encoder:BarrelJack_Horizontal (layer B.Cu)
+    (at 133.76148 139.25804 90)
     (descr "DC Barrel Jack")
     (tags "Power Jack")
-    (fp_text reference J4 (at -8.45 5.75 90) (layer F.SilkS)
-      (effects (font (size 1 1) (thickness 0.15)))
-    )
-    (fp_text value Barrel_Jack_Switch (at -6.2 -5.5 90) (layer F.Fab)
-      (effects (font (size 1 1) (thickness 0.15)))
-    )
-    (fp_text user %R (at -3 -2.95 90) (layer F.Fab)
-      (effects (font (size 1 1) (thickness 0.15)))
-    )
-    (fp_line (start -0.003213 -4.505425) (end 0.8 -3.75) (layer F.Fab) (width 0.1))
-    (fp_line (start 1.1 -3.75) (end 1.1 -4.8) (layer F.SilkS) (width 0.12))
-    (fp_line (start 0.05 -4.8) (end 1.1 -4.8) (layer F.SilkS) (width 0.12))
-    (fp_line (start 1 -4.5) (end 1 -4.75) (layer F.CrtYd) (width 0.05))
-    (fp_line (start 1 -4.75) (end -14 -4.75) (layer F.CrtYd) (width 0.05))
-    (fp_line (start 1 -4.5) (end 1 -2) (layer F.CrtYd) (width 0.05))
-    (fp_line (start 1 -2) (end 2 -2) (layer F.CrtYd) (width 0.05))
-    (fp_line (start 2 -2) (end 2 2) (layer F.CrtYd) (width 0.05))
-    (fp_line (start 2 2) (end 1 2) (layer F.CrtYd) (width 0.05))
-    (fp_line (start 1 2) (end 1 4.75) (layer F.CrtYd) (width 0.05))
-    (fp_line (start 1 4.75) (end -1 4.75) (layer F.CrtYd) (width 0.05))
-    (fp_line (start -1 4.75) (end -1 6.75) (layer F.CrtYd) (width 0.05))
-    (fp_line (start -1 6.75) (end -5 6.75) (layer F.CrtYd) (width 0.05))
-    (fp_line (start -5 6.75) (end -5 4.75) (layer F.CrtYd) (width 0.05))
-    (fp_line (start -5 4.75) (end -14 4.75) (layer F.CrtYd) (width 0.05))
-    (fp_line (start -14 4.75) (end -14 -4.75) (layer F.CrtYd) (width 0.05))
-    (fp_line (start -5 4.6) (end -13.8 4.6) (layer F.SilkS) (width 0.12))
-    (fp_line (start -13.8 4.6) (end -13.8 -4.6) (layer F.SilkS) (width 0.12))
-    (fp_line (start 0.9 1.9) (end 0.9 4.6) (layer F.SilkS) (width 0.12))
-    (fp_line (start 0.9 4.6) (end -1 4.6) (layer F.SilkS) (width 0.12))
-    (fp_line (start -13.8 -4.6) (end 0.9 -4.6) (layer F.SilkS) (width 0.12))
-    (fp_line (start 0.9 -4.6) (end 0.9 -2) (layer F.SilkS) (width 0.12))
-    (fp_line (start -10.2 -4.5) (end -10.2 4.5) (layer F.Fab) (width 0.1))
-    (fp_line (start -13.7 -4.5) (end -13.7 4.5) (layer F.Fab) (width 0.1))
-    (fp_line (start -13.7 4.5) (end 0.8 4.5) (layer F.Fab) (width 0.1))
-    (fp_line (start 0.8 4.5) (end 0.8 -3.75) (layer F.Fab) (width 0.1))
-    (fp_line (start 0 -4.5) (end -13.7 -4.5) (layer F.Fab) (width 0.1))
+    (fp_text reference J4 (at -8.45 -5.75 90) (layer B.SilkS)
+      (effects (font (size 1 1) (thickness 0.15)) (justify mirror))
+    )
+    (fp_text value Barrel_Jack_Switch (at -6.2 5.5 90) (layer B.Fab)
+      (effects (font (size 1 1) (thickness 0.15)) (justify mirror))
+    )
+    (fp_text user %R (at -3 2.95 90) (layer B.Fab)
+      (effects (font (size 1 1) (thickness 0.15)) (justify mirror))
+    )
+    (fp_line (start -0.003213 4.505425) (end 0.8 3.75) (layer B.Fab) (width 0.1))
+    (fp_line (start 1.1 3.75) (end 1.1 4.8) (layer B.SilkS) (width 0.12))
+    (fp_line (start 0.05 4.8) (end 1.1 4.8) (layer B.SilkS) (width 0.12))
+    (fp_line (start 1 4.5) (end 1 4.75) (layer B.CrtYd) (width 0.05))
+    (fp_line (start 1 4.75) (end -14 4.75) (layer B.CrtYd) (width 0.05))
+    (fp_line (start 1 4.5) (end 1 2) (layer B.CrtYd) (width 0.05))
+    (fp_line (start 1 2) (end 2 2) (layer B.CrtYd) (width 0.05))
+    (fp_line (start 2 2) (end 2 -2) (layer B.CrtYd) (width 0.05))
+    (fp_line (start 2 -2) (end 1 -2) (layer B.CrtYd) (width 0.05))
+    (fp_line (start 1 -2) (end 1 -4.75) (layer B.CrtYd) (width 0.05))
+    (fp_line (start 1 -4.75) (end -1 -4.75) (layer B.CrtYd) (width 0.05))
+    (fp_line (start -1 -4.75) (end -1 -6.75) (layer B.CrtYd) (width 0.05))
+    (fp_line (start -1 -6.75) (end -5 -6.75) (layer B.CrtYd) (width 0.05))
+    (fp_line (start -5 -6.75) (end -5 -4.75) (layer B.CrtYd) (width 0.05))
+    (fp_line (start -5 -4.75) (end -14 -4.75) (layer B.CrtYd) (width 0.05))
+    (fp_line (start -14 -4.75) (end -14 4.75) (layer B.CrtYd) (width 0.05))
+    (fp_line (start -5 -4.6) (end -13.8 -4.6) (layer B.SilkS) (width 0.12))
+    (fp_line (start -13.8 -4.6) (end -13.8 4.6) (layer B.SilkS) (width 0.12))
+    (fp_line (start 0.9 -1.9) (end 0.9 -4.6) (layer B.SilkS) (width 0.12))
+    (fp_line (start 0.9 -4.6) (end -1 -4.6) (layer B.SilkS) (width 0.12))
+    (fp_line (start -13.8 4.6) (end 0.9 4.6) (layer B.SilkS) (width 0.12))
+    (fp_line (start 0.9 4.6) (end 0.9 2) (layer B.SilkS) (width 0.12))
+    (fp_line (start -10.2 4.5) (end -10.2 -4.5) (layer B.Fab) (width 0.1))
+    (fp_line (start -13.7 4.5) (end -13.7 -4.5) (layer B.Fab) (width 0.1))
+    (fp_line (start -13.7 -4.5) (end 0.8 -4.5) (layer B.Fab) (width 0.1))
+    (fp_line (start 0.8 -4.5) (end 0.8 3.75) (layer B.Fab) (width 0.1))
+    (fp_line (start 0 4.5) (end -13.7 4.5) (layer B.Fab) (width 0.1))
     (pad 1 thru_hole rect (at 0 0 90) (size 3.5 3.5) (drill oval 1 3) (layers *.Cu *.Mask)
       (net 13 VCC))
     (pad 2 thru_hole roundrect (at -6 0 90) (size 3 3.5) (drill oval 1 3) (layers *.Cu *.Mask) (roundrect_rratio 0.25)
       (net 1 GND))
-    (pad 3 thru_hole roundrect (at -3 4.7 90) (size 3.5 3.5) (drill oval 3 1) (layers *.Cu *.Mask) (roundrect_rratio 0.25)
+    (pad 3 thru_hole roundrect (at -3 -4.7 90) (size 3.5 3.5) (drill oval 3 1) (layers *.Cu *.Mask) (roundrect_rratio 0.25)
       (net 1 GND))
     (model "${KIPRJMOD}/../FootPrints//3DModels/BarrelJack/DC Power Jack 5.5mm x 2.1mm.STEP"
@@
   (segment (start 111.167287 132.055376) (end 111.167287 131.618496) (width 0.635) (layer F.Cu) (net 13))
   (segment (start 112.449267 133.337356) (end 111.167287 132.055376) (width 0.635) (layer F.Cu) (net 13))
-  (segment (start 129.822 138.94816) (end 128.78308 139.98708) (width 1.27) (layer F.Cu) (net 13))
-  (segment (start 132.842 138.94816) (end 129.822 138.94816) (width 1.27) (layer F.Cu) (net 13))
-  (segment (start 128.78308 139.98708) (end 128.78308 142.06728) (width 1.27) (layer F.Cu) (net 13))
-  (segment (start 128.78308 142.06728) (end 125.41504 145.43532) (width 1.27) (layer F.Cu) (net 13))
   (segment (start 125.41504 145.43532) (end 118.9482 145.43532) (width 1.27) (layer F.Cu) (net 13))
   (segment (start 118.9482 145.43532) (end 116.40312 145.43532) (width 0.635) (layer F.Cu) (net 13))
@@
   (segment (start 114.010071 146.03476) (end 113.090067 145.114756) (width 0.635) (layer F.Cu) (net 13))
   (segment (start 115.80368 146.03476) (end 114.010071 146.03476) (width 0.635) (layer F.Cu) (net 13))
+  (segment (start 125.41504 145.43532) (end 130.19024 145.43532) (width 1.27) (layer F.Cu) (net 13))
+  (segment (start 130.19024 145.425908) (end 131.41452 144.201628) (width 0.635) (layer F.Cu) (net 13))
+  (segment (start 130.19024 145.43532) (end 130.19024 145.425908) (width 0.635) (layer F.Cu) (net 13))
+  (segment (start 131.41452 144.201628) (end 131.41452 143.16456) (width 0.635) (layer F.Cu) (net 13))
+  (segment (start 131.41452 143.16456) (end 132.68452 141.89456) (width 0.635) (layer F.Cu) (net 13))
+  (segment (start 133.76148 141.64304) (end 133.76148 139.25804) (width 0.635) (layer F.Cu) (net 13))
+  (segment (start 133.50996 141.89456) (end 133.76148 141.64304) (width 0.635) (layer F.Cu) (net 13))
+  (segment (start 132.68452 141.89456) (end 133.50996 141.89456) (width 0.635) (layer F.Cu) (net 13))
   (segment (start 124.44368 85.22016) (end 124.43968 85.21616) (width 0.1016) (layer F.Cu) (net 14))
   (segment (start 124.44368 86.10176) (end 124.44368 85.22016) (width 0.1016) (layer F.Cu) (net 14) (status 10))

Commit message: Added changes
Parts:
- J4: moved to F.Cu
- moved R13 63.0 mm to (111.1, 117.5), turned to 90 degrees
- moved R14 60.8 mm to (111.1, 114.2), turned to 90 degrees
- moved R5 26.6 mm to (121.3, 110.6)
- moved C8 20.7 mm to (108.8, 110.8), turned to 90 degrees
- moved C6 16.7 mm to (130.6, 99.7), turned to 270 degrees
- moved J1 16.4 mm to (134.4, 104.9), turned to 180 degrees
- moved C9 14.9 mm to (118.1, 99.5)
- moved C15 14.7 mm to (132.3, 86.5)
- moved C3 14.5 mm to (115.2, 109.2)
- moved C4 14.5 mm to (115.2, 110.8)
- moved R3 14.5 mm to (121.6, 119.1)
- moved Y1 14.5 mm to (110.1, 100.7)
- moved C10 14.5 mm to (127.6, 109.2)
- moved R4 14.5 mm to (133.3, 119.1)
- moved C1 14.5 mm to (115.2, 100.7)
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Connections:
- J1 pad 4: /RTS -> /F1TX
- J1 pad 5: /F1TX -> /F1RX
- J1 pad 6: /F1RX -> /RTS
- R13 pad 1: +3V3 -> /BattVolt
- R13 pad 2: /BattVolt -> Net-(R13-Pad2)
- R14 pad 1: /BattVolt -> Net-(R13-Pad2)
- R5 pad 2: Net-(R5-Pad2) -> /BOOT0
- U1 pad 11: /BattVolt -> Net-(R13-Pad2)
- U1 pad 20: (no net) -> /BOOT0
- U1 pad 22: Net-(IC1-Pad7) -> (no net)
- U1 pad 41: (no net) -> Net-(IC1-Pad7)
- U1 pad 44: Net-(R5-Pad2) -> /BOOT0
Routing:
- net +3V3: track 2.09 -> 179.1 mm
- net /F1TX: track 13.8 -> 32.9 mm
- net /F1RX: track 16.4 -> 34.3 mm
- net /BOOT0: track 0.00 -> 16.2 mm
- net Net-(R13-Pad2): track 0.00 -> 15.0 mm
- net Net-(C7-Pad2): track 0.00 -> 14.7 mm
- net Net-(C8-Pad2): track 0.00 -> 13.8 mm
- net Net-(IC1-Pad7): track 0.00 -> 11.3 mm
- net /CTS: track 0.00 -> 10.6 mm
- net /BattVolt: track 15.6 -> 25.9 mm
- net /SWCLK: track 0.64 -> 10.8 mm
- net /SWDIO: track 0.00 -> 8.19 mm
- net /RTS: track 0.00 -> 4.92 mm
- net Net-(C2-Pad1): track 0.00 -> 3.23 mm
- net /SIGA: track 25.0 -> 27.9 mm
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Other:
- board size 66 x 77.5 mm -> 66 x 63.5 mm

Commit message: Added changes
Parts:
- moved R9 1.23 mm to (121.9, 142.4)
- moved R5 0.94 mm to (120.4, 110.6)
- moved C2 0.81 mm to (114.8, 105.4)
Connections:
- R5 pad 1: +3V3 -> /BOOT0
- R5 pad 2: /BOOT0 -> GND
- U1 pad 20: /BOOT0 -> GND
Routing:
- net GND: track 0.01 -> 52.5 mm, vias 0 -> 33
- net /CHG: track 0.00 -> 44.9 mm, vias 0 -> 4
- net /STDBY: track 0.00 -> 44.3 mm, vias 0 -> 4
- net +3V3: track 179.1 -> 206.8 mm
- net /BOOT0: track 16.2 -> 11.2 mm
- net /SIGA: track 27.9 -> 29.9 mm
- net Net-(IC3-Pad1): track 15.3 -> 16.9 mm
- net Net-(IC3-Pad2): track 1.86 -> 3.09 mm
- net /F1TX: track 32.9 -> 34.1 mm
- net Net-(IC3-Pad3): track 10.8 -> 12.0 mm
- net Net-(IC1-Pad7): track 11.3 -> 12.4 mm
- net /F1RX: track 34.3 -> 35.3 mm
- net /SIGB: track 36.0 -> 36.7 mm
- added copper zone on B.Cu, net GND

Commit message: Added changes
Parts:
- added Q3: Q_PMOS_GSD, Encoder:SOT-23, F.Cu at (114.4, 116.4)
- moved R7 5.74 mm to (127.5, 127.8)
- moved C11 5.74 mm to (128.4, 131.3)
- moved C12 5.74 mm to (131.8, 131.3)
- moved C14 5.74 mm to (130.6, 126.5)
- moved U6 5.74 mm to (129.6, 129.0)
- moved R4 5.01 mm to (138.3, 119.4)
- moved U2 5.01 mm to (123.6, 114.8)
- moved R1 5.01 mm to (121.0, 119.4)
- moved R2 5.01 mm to (130.7, 119.3)
- moved R3 5.01 mm to (126.6, 119.4)
- moved U3 5.01 mm to (134.8, 114.9)
- turned S1 to 0 degrees
Connections:
- R3 pad 1: +3V3 -> Net-(Q3-Pad3)
- R4 pad 1: +3V3 -> Net-(Q3-Pad3)
- U1 pad 14: (no net) -> /EncEnable
- U2 pad 1: +3V3 -> Net-(Q3-Pad3)
- U3 pad 1: +3V3 -> Net-(Q3-Pad3)
Routing:
- net Net-(Q3-Pad3): track 0.00 -> 40.3 mm
- net +3V3: track 206.8 -> 187.0 mm
- net /EncEnable: track 0.00 -> 11.0 mm
- net /CHG: track 44.9 -> 55.7 mm
- net /STDBY: track 44.3 -> 54.3 mm
- net Net-(C11-Pad2): track 11.2 -> 17.0 mm
- net /SIGB: track 36.7 -> 36.1 mm
Other:
- board size 66 x 63.5 mm -> 37.8 x 63.5 mm

Commit message: Added changes
Parts:
- added C17: 10uF, Encoder:C_0603_1608Metric_Pad1.05x0.95mm_HandSolder, F.Cu at (125.3, 145.0)
- added D2: D, Encoder:D_SMA, F.Cu at (120.0, 144.5)
- moved J7 16.3 mm to (128.5, 141.9)
- moved J4 3.18 mm to (135.1, 139.3)
- moved IC3 1.09 mm to (120.7, 137.1)
- moved Q1 1.09 mm to (124.5, 137.0)
- moved R9 1.09 mm to (121.6, 141.4)
Connections:
- net /BattVolt renamed /Batt+
- net Net-(C16-Pad2) renamed GNDPWR
Routing:
- net GNDPWR: track 15.1 -> 38.0 mm
- net VCC: track 59.5 -> 69.2 mm
- net Net-(C16-Pad1): track 9.98 -> 9.13 mm
- net Net-(IC3-Pad1): track 16.9 -> 16.1 mm

Commit message: Added changes
Parts:
- added J2: VCC, Encoder:No3dmodelPinHeader_1x01_P2.54mm_Vertical, F.Cu at (135.5, 144.5)
- added J3: GND, Encoder:No3dmodelPinHeader_1x01_P2.54mm_Vertical, F.Cu at (139.2, 144.5)
- J4: value Barrel_Jack_Switch -> GND; footprint Encoder:BarrelJack_Horizontal -> Encoder:No3dmodelPinHeader_1x01_P2.54mm_Vertical
- moved J4 4.34 mm to (139.2, 140.9)
Connections:
- J4 pad 1: VCC -> GND
Routing:
- net /SIGA: track 30.3 -> 23.0 mm
- net VCC: track 69.2 -> 65.9 mm
