File: Mechatronics/Hardware/Electrical/BEncoderBoard/EncoderBoard.kicad_pcb (KiCad board)
At the start: 2 copper layers, 37.8 x 63.5 mm, 50 parts, among them IC1 RN4020-V_RM120, IC2 TP4056, IC3 DW01+G, J1 Conn_01x07_Male, J2 VCC, J3 GND, J4 GND, J5 Batt+, J7 Batt-, Q1 FS8205, Q2 Q_PMOS_GSD, Q3 Q_PMOS_GSD, U1 STM32F103C8T6, U2 ITR1802A, U3 ITR1802B, U5 SSD1306OLED, U6 LTC2430, Y1 8Mhz

Commit message: Added changes
Parts:
- removed J2: VCC, Encoder:No3dmodelPinHeader_1x01_P2.54mm_Vertical
- removed J3: GND, Encoder:No3dmodelPinHeader_1x01_P2.54mm_Vertical
- J4: value GND -> Barrel_Jack_Switch; footprint Encoder:No3dmodelPinHeader_1x01_P2.54mm_Vertical -> Encoder:BarrelJack_Horizontal
- moved J4 4.50 mm to (135.0, 139.2)
Connections:
- J4 pad 1: GND -> VCC
Routing:
- net VCC: track 65.9 -> 68.1 mm
- net GND: track 52.3 -> 53.8 mm
Changed lines of the file:
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@@
     (thickness 1.6)
     (drawings 8)
-    (tracks 576)
+    (tracks 577)
     (zones 0)
-    (modules 50)
+    (modules 48)
     (nets 38)
   )
@@
     )
   )
-  (module Encoder:No3dmodelPinHeader_1x01_P2.54mm_Vertical (layer F.Cu)
-    (at 135.530601 144.522201)
-    (descr "Through hole straight pin header, 1x01, 2.54mm pitch, single row")
-    (tags "Through hole pin header THT 1x01 2.54mm single row")
-    (fp_text reference J2 (at 0 -2.33) (layer F.SilkS) hide
-      (effects (font (size 1 1) (thickness 0.15)))
-    )
-    (fp_text value VCC (at 0 2.33) (layer F.Fab)
-      (effects (font (size 1 1) (thickness 0.15)))
-    )
-    (fp_text user %R (at 0 0 90) (layer F.Fab)
-      (effects (font (size 1 1) (thickness 0.15)))
-    )
-    (fp_line (start 1.8 -1.8) (end -1.8 -1.8) (layer F.CrtYd) (width 0.05))
-    (fp_line (start 1.8 1.8) (end 1.8 -1.8) (layer F.CrtYd) (width 0.05))
-    (fp_line (start -1.8 1.8) (end 1.8 1.8) (layer F.CrtYd) (width 0.05))
-    (fp_line (start -1.8 -1.8) (end -1.8 1.8) (layer F.CrtYd) (width 0.05))
-    (fp_line (start -1.27 -0.635) (end -0.635 -1.27) (layer F.Fab) (width 0.1))
-    (fp_line (start -1.27 1.27) (end -1.27 -0.635) (layer F.Fab) (width 0.1))
-    (fp_line (start 1.27 1.27) (end -1.27 1.27) (layer F.Fab) (width 0.1))
-    (fp_line (start 1.27 -1.27) (end 1.27 1.27) (layer F.Fab) (width 0.1))
-    (fp_line (start -0.635 -1.27) (end 1.27 -1.27) (layer F.Fab) (width 0.1))
-    (pad 1 thru_hole rect (at 0 0) (size 1.7 1.7) (drill 1) (layers *.Cu *.Mask)
+  (module Encoder:BarrelJack_Horizontal (layer F.Cu)
+    (at 134.9756 139.2428 90)
+    (descr "DC Barrel Jack")
+    (tags "Power Jack")
+    (fp_text reference J4 (at -8.45 5.75 90) (layer F.SilkS)
+      (effects (font (size 1 1) (thickness 0.15)))
+    )
+    (fp_text value Barrel_Jack_Switch (at -6.2 -5.5 90) (layer F.Fab)
+      (effects (font (size 1 1) (thickness 0.15)))
+    )
+    (fp_text user %R (at -3 -2.95 90) (layer F.Fab)
+      (effects (font (size 1 1) (thickness 0.15)))
+    )
+    (fp_line (start -0.003213 -4.505425) (end 0.8 -3.75) (layer F.Fab) (width 0.1))
+    (fp_line (start 1.1 -3.75) (end 1.1 -4.8) (layer F.SilkS) (width 0.12))
+    (fp_line (start 0.05 -4.8) (end 1.1 -4.8) (layer F.SilkS) (width 0.12))
+    (fp_line (start 1 -4.5) (end 1 -4.75) (layer F.CrtYd) (width 0.05))
+    (fp_line (start 1 -4.75) (end -14 -4.75) (layer F.CrtYd) (width 0.05))
+    (fp_line (start 1 -4.5) (end 1 -2) (layer F.CrtYd) (width 0.05))
+    (fp_line (start 1 -2) (end 2 -2) (layer F.CrtYd) (width 0.05))
+    (fp_line (start 2 -2) (end 2 2) (layer F.CrtYd) (width 0.05))
+    (fp_line (start 2 2) (end 1 2) (layer F.CrtYd) (width 0.05))
+    (fp_line (start 1 2) (end 1 4.75) (layer F.CrtYd) (width 0.05))
+    (fp_line (start 1 4.75) (end -1 4.75) (layer F.CrtYd) (width 0.05))
+    (fp_line (start -1 4.75) (end -1 6.75) (layer F.CrtYd) (width 0.05))
+    (fp_line (start -1 6.75) (end -5 6.75) (layer F.CrtYd) (width 0.05))
+    (fp_line (start -5 6.75) (end -5 4.75) (layer F.CrtYd) (width 0.05))
+    (fp_line (start -5 4.75) (end -14 4.75) (layer F.CrtYd) (width 0.05))
+    (fp_line (start -14 4.75) (end -14 -4.75) (layer F.CrtYd) (width 0.05))
+    (fp_line (start -5 4.6) (end -13.8 4.6) (layer F.SilkS) (width 0.12))
+    (fp_line (start -13.8 4.6) (end -13.8 -4.6) (layer F.SilkS) (width 0.12))
+    (fp_line (start 0.9 1.9) (end 0.9 4.6) (layer F.SilkS) (width 0.12))
+    (fp_line (start 0.9 4.6) (end -1 4.6) (layer F.SilkS) (width 0.12))
+    (fp_line (start -13.8 -4.6) (end 0.9 -4.6) (layer F.SilkS) (width 0.12))
+    (fp_line (start 0.9 -4.6) (end 0.9 -2) (layer F.SilkS) (width 0.12))
+    (fp_line (start -10.2 -4.5) (end -10.2 4.5) (layer F.Fab) (width 0.1))
+    (fp_line (start -13.7 -4.5) (end -13.7 4.5) (layer F.Fab) (width 0.1))
+    (fp_line (start -13.7 4.5) (end 0.8 4.5) (layer F.Fab) (width 0.1))
+    (fp_line (start 0.8 4.5) (end 0.8 -3.75) (layer F.Fab) (width 0.1))
+    (fp_line (start 0 -4.5) (end -13.7 -4.5) (layer F.Fab) (width 0.1))
+    (pad 1 thru_hole rect (at 0 0 90) (size 3.5 3.5) (drill oval 1 3) (layers *.Cu *.Mask)
       (net 13 VCC))
-    (model ${KISYS3DMOD}/Connector_PinHeader_2.54mm.3dshapes/PinHeader_1x01_P2.54mm_Vertical.wrl
-      (at (xyz 0 0 0))
-      (scale (xyz 1 1 1))
-      (rotate (xyz 0 0 0))
-    )
-  )
-  (module Encoder:No3dmodelPinHeader_1x01_P2.54mm_Vertical (layer F.Cu)
-    (at 139.180601 144.522201)
-    (descr "Through hole straight pin header, 1x01, 2.54mm pitch, single row")
-    (tags "Through hole pin header THT 1x01 2.54mm single row")
-    (fp_text reference J3 (at 0 -2.33) (layer F.SilkS) hide
-      (effects (font (size 1 1) (thickness 0.15)))
-    )
-    (fp_text value GND (at 0 2.33) (layer F.Fab)
-      (effects (font (size 1 1) (thickness 0.15)))
-    )
-    (fp_line (start -0.635 -1.27) (end 1.27 -1.27) (layer F.Fab) (width 0.1))
-    (fp_line (start 1.27 -1.27) (end 1.27 1.27) (layer F.Fab) (width 0.1))
-    (fp_line (start 1.27 1.27) (end -1.27 1.27) (layer F.Fab) (width 0.1))
-    (fp_line (start -1.27 1.27) (end -1.27 -0.635) (layer F.Fab) (width 0.1))
-    (fp_line (start -1.27 -0.635) (end -0.635 -1.27) (layer F.Fab) (width 0.1))
-    (fp_line (start -1.8 -1.8) (end -1.8 1.8) (layer F.CrtYd) (width 0.05))
-    (fp_line (start -1.8 1.8) (end 1.8 1.8) (layer F.CrtYd) (width 0.05))
-    (fp_line (start 1.8 1.8) (end 1.8 -1.8) (layer F.CrtYd) (width 0.05))
-    (fp_line (start 1.8 -1.8) (end -1.8 -1.8) (layer F.CrtYd) (width 0.05))
-    (fp_text user %R (at 0 0 90) (layer F.Fab)
-      (effects (font (size 1 1) (thickness 0.15)))
-    )
-    (pad 1 thru_hole rect (at 0 0) (size 1.7 1.7) (drill 1) (layers *.Cu *.Mask)
-      (net 1 GND))
-    (model ${KISYS3DMOD}/Connector_PinHeader_2.54mm.3dshapes/PinHeader_1x01_P2.54mm_Vertical.wrl
-      (at (xyz 0 0 0))
-      (scale (xyz 1 1 1))
-      (rotate (xyz 0 0 0))
-    )
-  )
-  (module Encoder:No3dmodelPinHeader_1x01_P2.54mm_Vertical (layer F.Cu)
-    (at 139.1666 140.8938 90)
-    (descr "Through hole straight pin header, 1x01, 2.54mm pitch, single row")
-    (tags "Through hole pin header THT 1x01 2.54mm single row")
-    (fp_text reference J4 (at 0 -2.33 90) (layer F.SilkS) hide
-      (effects (font (size 1 1) (thickness 0.15)))
-    )
-    (fp_text value GND (at 0 2.33 90) (layer F.Fab)
-      (effects (font (size 1 1) (thickness 0.15)))
-    )
-    (fp_line (start -0.635 -1.27) (end 1.27 -1.27) (layer F.Fab) (width 0.1))
-    (fp_line (start 1.27 -1.27) (end 1.27 1.27) (layer F.Fab) (width 0.1))
-    (fp_line (start 1.27 1.27) (end -1.27 1.27) (layer F.Fab) (width 0.1))
-    (fp_line (start -1.27 1.27) (end -1.27 -0.635) (layer F.Fab) (width 0.1))
-    (fp_line (start -1.27 -0.635) (end -0.635 -1.27) (layer F.Fab) (width 0.1))
-    (fp_line (start -1.8 -1.8) (end -1.8 1.8) (layer F.CrtYd) (width 0.05))
-    (fp_line (start -1.8 1.8) (end 1.8 1.8) (layer F.CrtYd) (width 0.05))
-    (fp_line (start 1.8 1.8) (end 1.8 -1.8) (layer F.CrtYd) (width 0.05))
-    (fp_line (start 1.8 -1.8) (end -1.8 -1.8) (layer F.CrtYd) (width 0.05))
-    (fp_text user %R (at 0 0 180) (layer F.Fab)
-      (effects (font (size 1 1) (thickness 0.15)))
-    )
-    (pad 1 thru_hole rect (at 0 0 90) (size 1.7 1.7) (drill 1) (layers *.Cu *.Mask)
-      (net 1 GND))
-    (model ${KISYS3DMOD}/Connector_PinHeader_2.54mm.3dshapes/PinHeader_1x01_P2.54mm_Vertical.wrl
-      (at (xyz 0 0 0))
-      (scale (xyz 1 1 1))
-      (rotate (xyz 0 0 0))
+    (pad 2 thru_hole roundrect (at -6 0 90) (size 3 3.5) (drill oval 1 3) (layers *.Cu *.Mask) (roundrect_rratio 0.25)
+      (net 1 GND))
+    (pad 3 thru_hole roundrect (at -3 4.7 90) (size 3.5 3.5) (drill oval 3 1) (layers *.Cu *.Mask) (roundrect_rratio 0.25)
+      (net 1 GND))
+    (model "${KIPRJMOD}/../FootPrints//3DModels/BarrelJack/DC Power Jack 5.5mm x 2.1mm.STEP"
+      (offset (xyz -10.75 0 6))
+      (scale (xyz 1 1 1))
+      (rotate (xyz -90 0 90))
     )
   )
@@
   (segment (start 118.639 146.7104) (end 118.9736 146.7104) (width 0.635) (layer F.Cu) (net 13))
   (segment (start 118.9736 146.7104) (end 122.682 146.7104) (width 0.635) (layer F.Cu) (net 13))
-  (segment (start 134.827402 146.7104) (end 135.530601 146.007201) (width 0.635) (layer F.Cu) (net 13))
-  (segment (start 135.530601 146.007201) (end 135.530601 144.522201) (width 0.635) (layer F.Cu) (net 13))
-  (segment (start 127.3 146.7104) (end 134.827402 146.7104) (width 0.635) (layer F.Cu) (net 13))
+  (segment (start 135.530601 146.007201) (end 135.530601 144.522201) (width 0.635) (layer F.Cu) (net 1))
+  (segment (start 134.9756 141.6278) (end 134.9756 139.2428) (width 0.635) (layer F.Cu) (net 13))
+  (segment (start 129.893 146.7104) (end 134.9756 141.6278) (width 0.635) (layer F.Cu) (net 13))
+  (segment (start 127.3 146.7104) (end 129.893 146.7104) (width 0.635) (layer F.Cu) (net 13))
   (segment (start 115.9637 90.25636) (end 116.2962 89.92386) (width 0.254) (layer F.Cu) (net 14))
   (segment (start 116.2962 89.92386) (end 118.0242 89.92386) (width 0.254) (layer F.Cu) (net 14) (status 20))

Commit message: Added changes
Parts:
- removed D2: D, Encoder:D_SMA
- added C18: 1uF, Encoder:C_0603_1608Metric_Pad1.05x0.95mm_HandSolder, F.Cu at (127.7, 145.1)
- added U4: 82402305, Encoder:Sot-23(6), F.Cu at (119.7, 144.5)
- C17: value 10uF -> 1uF
- moved C17 1.17 mm to (124.1, 145.1)
Connections:
- IC3 pad 3: Net-(IC3-Pad3) -> (no net)
- Q1 pad 1: GND -> (no net)
- Q1 pad 5: (no net) -> GND
- Q1 pad 6: Net-(IC3-Pad3) -> (no net)
Routing:
- net Net-(IC3-Pad3): track 12.0 -> 0.00 mm
- net /SIGA: track 23.0 -> 30.3 mm
- net VCC: track 68.1 -> 70.8 mm
- net GNDPWR: track 38.0 -> 39.4 mm
- net GND: track 53.8 -> 55.0 mm

Commit message: Added changes
Parts:
- added J2: GNDPWR, Encoder:No3dmodelPinHeader_1x01_P2.54mm_Vertical, F.Cu at (128.2, 142.2)
- U6: value LTC2430 -> LTC3240
- moved J7 16.3 mm to (116.3, 131.2)
Connections:
- C16 pad 2: GNDPWR -> GND
- C17 pad 2: GNDPWR -> GND
- C18 pad 2: GNDPWR -> GND
- IC3 pad 6: GNDPWR -> GND
- J7 pad 1: GNDPWR -> GND
- Q1 pad 3: GNDPWR -> GND
- U4 pad 2: GNDPWR -> GND
Routing:
- net GND: track 55.0 -> 98.2 mm
- net GNDPWR: track 39.4 -> 0.00 mm

Commit message: Added changes
Connections:
- IC2 pad 6: /STDBY -> (no net)
- IC2 pad 7: /CHG -> (no net)
- IC3 pad 3: (no net) -> Net-(IC3-Pad3)
- Q1 pad 1: (no net) -> GND
- Q1 pad 5: GND -> (no net)
- Q1 pad 6: (no net) -> Net-(IC3-Pad3)
- U1 pad 25: /CHG -> VCC
- U1 pad 26: /STDBY -> (no net)
Routing:
- net /CHG: track 55.7 -> 0.00 mm, vias 4 -> 0
- net /STDBY: track 54.3 -> 0.00 mm, vias 4 -> 0
- net VCC: track 70.8 -> 115.0 mm, vias 0 -> 4
- net Net-(IC3-Pad3): track 0.00 -> 11.8 mm
- net GND: track 98.2 -> 95.4 mm
