File: Mechatronics/Hardware/Electrical/BEncoderBoard/EncoderBoard.kicad_pcb (KiCad board)
At the start: 2 copper layers, 37.8 x 63.5 mm, 50 parts, among them IC1 RN4020-V_RM120, IC2 TP4056, IC3 DW01+G, J1 Conn_01x07_Male, J2 GNDPWR, J4 Barrel_Jack_Switch, J5 Batt+, J7 Batt-, Q1 FS8205, Q2 Q_PMOS_GSD, Q3 Q_PMOS_GSD, U1 STM32F103C8T6, U2 ITR1802A, U3 ITR1802B, U4 82402305, U5 SSD1306OLED, U6 LTC3240, Y1 8Mhz

Commit message: Added changes
Parts:
- added D2: D, Diode_THT:D_DO-201AD_P5.08mm_Vertical_AnodeUp, F.Cu at (135.0, 134.3)
- U2: value ITR1802A -> ITR1802
- U3: value ITR1802B -> ITR1802
Connections:
- IC1 pad 10: (no net) -> Net-(IC1-Pad10)
- IC1 pad 11: (no net) -> Net-(IC1-Pad11)
- IC1 pad 12: (no net) -> Net-(IC1-Pad12)
- IC1 pad 13: (no net) -> Net-(IC1-Pad13)
- IC1 pad 15: (no net) -> Net-(IC1-Pad15)
- IC1 pad 17: (no net) -> Net-(IC1-Pad17)
- IC1 pad 19: (no net) -> Net-(IC1-Pad19)
- IC1 pad 2: (no net) -> Net-(IC1-Pad2)
- IC1 pad 20: (no net) -> Net-(IC1-Pad20)
- IC1 pad 21: (no net) -> Net-(IC1-Pad21)
- IC1 pad 22: (no net) -> Net-(IC1-Pad22)
- IC1 pad 3: (no net) -> Net-(IC1-Pad3)
- IC1 pad 4: (no net) -> Net-(IC1-Pad4)
- IC1 pad 8: (no net) -> Net-(IC1-Pad8)
- IC2 pad 6: (no net) -> Net-(IC2-Pad6)
- IC2 pad 7: (no net) -> Net-(IC2-Pad7)
- IC2 pad 9: (no net) -> Net-(IC2-Pad9)
- IC3 pad 4: (no net) -> Net-(IC3-Pad4)
- Q1 pad 2: (no net) -> Net-(Q1-Pad2)
- Q1 pad 5: (no net) -> Net-(Q1-Pad5)
- U1 pad 10: (no net) -> Net-(U1-Pad10)
- U1 pad 12: (no net) -> Net-(U1-Pad12)
- U1 pad 13: (no net) -> Net-(U1-Pad13)
- U1 pad 15: (no net) -> Net-(U1-Pad15)
- U1 pad 16: (no net) -> Net-(U1-Pad16)
- U1 pad 17: (no net) -> Net-(U1-Pad17)
- U1 pad 18: (no net) -> Net-(U1-Pad18)
- U1 pad 19: (no net) -> Net-(U1-Pad19)
- U1 pad 2: (no net) -> Net-(U1-Pad2)
- U1 pad 21: (no net) -> Net-(U1-Pad21)
- U1 pad 22: (no net) -> Net-(U1-Pad22)
- U1 pad 26: (no net) -> Net-(U1-Pad26)
- U1 pad 27: (no net) -> Net-(U1-Pad27)
- U1 pad 28: (no net) -> Net-(U1-Pad28)
- U1 pad 3: (no net) -> Net-(U1-Pad3)
- U1 pad 30: (no net) -> Net-(U1-Pad30)
- U1 pad 32: (no net) -> Net-(U1-Pad32)
- U1 pad 33: (no net) -> Net-(U1-Pad33)
- U1 pad 4: (no net) -> Net-(U1-Pad4)
- U1 pad 40: (no net) -> Net-(U1-Pad40)

Commit message: Added changes
Parts:
- removed D2: D, Diode_THT:D_DO-201AD_P5.08mm_Vertical_AnodeUp
- Q1: value FS8205 -> DMosfet
- moved C8 0.13 mm to (108.9, 110.9)
Connections:
- U4 pad 1: (no net) -> Net-(U4-Pad1)
- U4 pad 3: (no net) -> Net-(U4-Pad3)
- U4 pad 4: (no net) -> Net-(U4-Pad4)
- U4 pad 6: (no net) -> Net-(U4-Pad6)
Changed lines of the file:
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@@
     (tracks 560)
     (zones 0)
-    (modules 51)
-    (nets 75)
+    (modules 50)
+    (nets 79)
   )
   (page USLetter)
@@
   (net 73 "Net-(U1-Pad3)")
   (net 74 "Net-(U1-Pad2)")
+  (net 75 "Net-(U4-Pad6)")
+  (net 76 "Net-(U4-Pad4)")
+  (net 77 "Net-(U4-Pad3)")
+  (net 78 "Net-(U4-Pad1)")
   (net_class Default "Esta es la clase de red por defecto."
     (clearance 0.1016)
@@
     (add_net "Net-(U1-Pad4)")
     (add_net "Net-(U1-Pad40)")
+    (add_net "Net-(U4-Pad1)")
+    (add_net "Net-(U4-Pad3)")
+    (add_net "Net-(U4-Pad4)")
+    (add_net "Net-(U4-Pad6)")
     (add_net VCC)
   )
@@
   )
   (module Encoder:C_0603_1608Metric_Pad1.05x0.95mm_HandSolder (layer F.Cu)
-    (at 108.79836 110.75416 90)
+    (at 108.8644 110.871 90)
     (descr "Capacitor SMD 0603 (1608 Metric), square (rectangular) end terminal, IPC_7351 nominal with elongated pad for handsoldering. (Body size source: http://www.tortai-tech.com/upload/download/2011102023233369053.pdf), generated with kicad-footprint-generator")
     (tags "capacitor handsolder")
@@
     (attr smd)
     (fp_text reference IC3 (at -2.897364 -0.021967 180) (layer F.SilkS)
-      (effects (font (size 1.27 1.27) (thickness 0.254)))
+      (effects (font (size 1 1) (thickness 0.15)))
     )
     (fp_text value DW01+G (at 0 0 90) (layer F.SilkS) hide
@@
       (scale (xyz 1 1 1))
       (rotate (xyz 0 0 90))
-    )
-  )
-  (module "Encoder:Sot-23(6)" (layer F.Cu)
-    (at 124.451487 137.013456 90)
-    (descr sot-23-6,)
-    (tags "Integrated Circuit")
-    (attr smd)
-    (fp_text reference Q1 (at -0.019544 3.056513 180) (layer F.SilkS)
-      (effects (font (size 1.27 1.27) (thickness 0.254)))
-    )
-    (fp_text value FS8205 (at 0 0 90) (layer F.SilkS) hide
-      (effects (font (size 1.27 1.27) (thickness 0.254)))
-    )
-    (fp_line (start -1.85 -1.6) (end -0.65 -1.6) (layer F.SilkS) (width 0.2))
-    (fp_line (start -0.3 1.45) (end -0.3 -1.45) (layer F.SilkS) (width 0.2))
-    (fp_line (start 0.3 1.45) (end -0.3 1.45) (layer F.SilkS) (width 0.2))
-    (fp_line (start 0.3 -1.45) (end 0.3 1.45) (layer F.SilkS) (width 0.2))
-    (fp_line (start -0.3 -1.45) (end 0.3 -1.45) (layer F.SilkS) (width 0.2))
-    (fp_line (start -0.8 -0.5) (end 0.15 -1.45) (layer F.Fab) (width 0.1))
-    (fp_line (start -0.8 1.45) (end -0.8 -1.45) (layer F.Fab) (width 0.1))
-    (fp_line (start 0.8 1.45) (end -0.8 1.45) (layer F.Fab) (width 0.1))
-    (fp_line (start 0.8 -1.45) (end 0.8 1.45) (layer F.Fab) (width 0.1))
-    (fp_line (start -0.8 -1.45) (end 0.8 -1.45) (layer F.Fab) (width 0.1))
-    (fp_line (start -2.1 1.775) (end -2.1 -1.775) (layer F.CrtYd) (width 0.05))
-    (fp_line (start 2.1 1.775) (end -2.1 1.775) (layer F.CrtYd) (width 0.05))
-    (fp_line (start 2.1 -1.775) (end 2.1 1.775) (layer F.CrtYd) (width 0.05))
-    (fp_line (start -2.1 -1.775) (end 2.1 -1.775) (layer F.CrtYd) (width 0.05))
-    (fp_text user %R (at 0 0 90) (layer F.Fab)
-      (effects (font (size 1.27 1.27) (thickness 0.254)))
-    )
-    (pad 6 smd rect (at 1.25 -0.95 180) (size 0.6 1.2) (layers F.Cu F.Paste F.Mask)
-      (net 34 "Net-(IC3-Pad3)"))
-    (pad 5 smd rect (at 1.25 0 180) (size 0.6 1.2) (layers F.Cu F.Paste F.Mask)
-      (net 53 "Net-(Q1-Pad5)"))
-    (pad 4 smd rect (at 1.25 0.95 180) (size 0.6 1.2) (layers F.Cu F.Paste F.Mask)
-      (net 27 "Net-(IC3-Pad1)"))
-    (pad 3 smd rect (at -1.25 0.95 180) (size 0.6 1.2) (layers F.Cu F.Paste F.Mask)
-      (net 1 GND))
-    (pad 2 smd rect (at -1.25 0 180) (size 0.6 1.2) (layers F.Cu F.Paste F.Mask)
-      (net 54 "Net-(Q1-Pad2)"))
-    (pad 1 smd rect (at -1.25 -0.95 180) (size 0.6 1.2) (layers F.Cu F.Paste F.Mask)
-      (net 1 GND))
-    (model "${KIPRJMOD}/../FootPrints/3DModels/Sot23(6)/SOT23-6.stp"
-      (at (xyz 0 0 0))
-      (scale (xyz 1 1 1))
-      (rotate (xyz 0 0 0))
     )
   )
@@
     (tags "Integrated Circuit")
     (attr smd)
-    (fp_text reference U4 (at 0 0) (layer F.SilkS)
-      (effects (font (size 1.27 1.27) (thickness 0.254)))
+    (fp_text reference U4 (at 0.0508 -2.1082) (layer F.SilkS)
+      (effects (font (size 1 1) (thickness 0.15)))
     )
     (fp_text value 82402305 (at 0 0 180) (layer F.SilkS) hide
@@
       (effects (font (size 1.27 1.27) (thickness 0.254)))
     )
-    (pad 6 smd rect (at 1.25 -0.95 270) (size 0.6 1.2) (layers F.Cu F.Paste F.Mask))
+    (pad 6 smd rect (at 1.25 -0.95 270) (size 0.6 1.2) (layers F.Cu F.Paste F.Mask)
+      (net 75 "Net-(U4-Pad6)"))
     (pad 5 smd rect (at 1.25 0 270) (size 0.6 1.2) (layers F.Cu F.Paste F.Mask)
       (net 13 VCC))
-    (pad 4 smd rect (at 1.25 0.95 270) (size 0.6 1.2) (layers F.Cu F.Paste F.Mask))
-    (pad 3 smd rect (at -1.25 0.95 270) (size 0.6 1.2) (layers F.Cu F.Paste F.Mask))
+    (pad 4 smd rect (at 1.25 0.95 270) (size 0.6 1.2) (layers F.Cu F.Paste F.Mask)
+      (net 76 "Net-(U4-Pad4)"))
+    (pad 3 smd rect (at -1.25 0.95 270) (size 0.6 1.2) (layers F.Cu F.Paste F.Mask)
+      (net 77 "Net-(U4-Pad3)"))
     (pad 2 smd rect (at -1.25 0 270) (size 0.6 1.2) (layers F.Cu F.Paste F.Mask)
       (net 1 GND))
-    (pad 1 smd rect (at -1.25 -0.95 270) (size 0.6 1.2) (layers F.Cu F.Paste F.Mask))
+    (pad 1 smd rect (at -1.25 -0.95 270) (size 0.6 1.2) (layers F.Cu F.Paste F.Mask)
+      (net 78 "Net-(U4-Pad1)"))
     (model "${KIPRJMOD}/../FootPrints/3DModels/Sot23(6)/SOT23-6.stp"
       (at (xyz 0 0 0))
@@
       (net 1 GND))
   )
-  (module Diode_THT:D_DO-201AD_P5.08mm_Vertical_AnodeUp (layer F.Cu)
-    (at 134.9756 134.3152)
-    (descr "Diode, DO-201AD series, Axial, Vertical, pin pitch=5.08mm, , length*diameter=9.5*5.2mm^2, , http://www.diodes.com/_files/packages/DO-201AD.pdf")
-    (tags "Diode DO-201AD series Axial Vertical pin pitch 5.08mm  length 9.5mm diameter 5.2mm")
-    (fp_text reference D2 (at 2.54 -3.72) (layer F.SilkS)
-      (effects (font (size 1 1) (thickness 0.15)))
-    )
-    (fp_text value D (at 2.54 5.498) (layer F.Fab)
-      (effects (font (size 1 1) (thickness 0.15)))
-    )
-    (fp_circle (center 0 0) (end 2.6 0) (layer F.Fab) (width 0.1))
-    (fp_circle (center 0 0) (end 2.72 0) (layer F.SilkS) (width 0.12))
-    (fp_line (start 0 0) (end 5.08 0) (layer F.Fab) (width 0.1))
-    (fp_line (start 2.72 0) (end 3.18 0) (layer F.SilkS) (width 0.12))
-    (fp_line (start -2.85 -2.85) (end -2.85 2.85) (layer F.CrtYd) (width 0.05))
-    (fp_line (start -2.85 2.85) (end 6.93 2.85) (layer F.CrtYd) (width 0.05))
-    (fp_line (start 6.93 2.85) (end 6.93 -2.85) (layer F.CrtYd) (width 0.05))
-    (fp_line (start 6.93 -2.85) (end -2.85 -2.85) (layer F.CrtYd) (width 0.05))
-    (fp_text user %R (at 2.54 -3.72) (layer F.Fab)
-      (effects (font (size 1 1) (thickness 0.15)))
-    )
-    (fp_text user A (at 5.08 2.6) (layer F.Fab)
-      (effects (font (size 1 1) (thickness 0.15)))
-    )
-    (fp_text user A (at 5.08 2.6) (layer F.SilkS)
-      (effects (font (size 1 1) (thickness 0.15)))
-    )
-    (pad 1 thru_hole rect (at 0 0) (size 3.2 3.2) (drill 1.6) (layers *.Cu *.Mask)
-      (net 13 VCC))
-    (pad 2 thru_hole oval (at 5.08 0) (size 3.2 3.2) (drill 1.6) (layers *.Cu *.Mask)
-      (net 1 GND))
-    (model ${KISYS3DMOD}/Diode_THT.3dshapes/D_DO-201AD_P5.08mm_Vertical_AnodeUp.wrl
-      (at (xyz 0 0 0))
-      (scale (xyz 1 1 1))
+  (module "Encoder:Sot-23(6)" (layer F.Cu)
+    (at 124.46 137.0584 90)
+    (descr sot-23-6,)
+    (tags "Integrated Circuit")
+    (attr smd)
+    (fp_text reference Q1 (at 0.0508 2.4892 90) (layer F.SilkS)
+      (effects (font (size 1 1) (thickness 0.15)))
+    )
+    (fp_text value DMosfet (at 0 0 90) (layer F.SilkS) hide
+      (effects (font (size 1.27 1.27) (thickness 0.254)))
+    )
+    (fp_text user %R (at 0 0 90) (layer F.Fab)
+      (effects (font (size 1.27 1.27) (thickness 0.254)))
+    )
+    (fp_line (start -2.1 -1.775) (end 2.1 -1.775) (layer F.CrtYd) (width 0.05))
+    (fp_line (start 2.1 -1.775) (end 2.1 1.775) (layer F.CrtYd) (width 0.05))
+    (fp_line (start 2.1 1.775) (end -2.1 1.775) (layer F.CrtYd) (width 0.05))
+    (fp_line (start -2.1 1.775) (end -2.1 -1.775) (layer F.CrtYd) (width 0.05))
+    (fp_line (start -0.8 -1.45) (end 0.8 -1.45) (layer F.Fab) (width 0.1))
+    (fp_line (start 0.8 -1.45) (end 0.8 1.45) (layer F.Fab) (width 0.1))
+    (fp_line (start 0.8 1.45) (end -0.8 1.45) (layer F.Fab) (width 0.1))
+    (fp_line (start -0.8 1.45) (end -0.8 -1.45) (layer F.Fab) (width 0.1))
+    (fp_line (start -0.8 -0.5) (end 0.15 -1.45) (layer F.Fab) (width 0.1))
+    (fp_line (start -0.3 -1.45) (end 0.3 -1.45) (layer F.SilkS) (width 0.2))
+    (fp_line (start 0.3 -1.45) (end 0.3 1.45) (layer F.SilkS) (width 0.2))
+    (fp_line (start 0.3 1.45) (end -0.3 1.45) (layer F.SilkS) (width 0.2))
+    (fp_line (start -0.3 1.45) (end -0.3 -1.45) (layer F.SilkS) (width 0.2))
+    (fp_line (start -1.85 -1.6) (end -0.65 -1.6) (layer F.SilkS) (width 0.2))
+    (pad 1 smd rect (at -1.25 -0.95 180) (size 0.6 1.2) (layers F.Cu F.Paste F.Mask)
+      (net 1 GND))
+    (pad 2 smd rect (at -1.25 0 180) (size 0.6 1.2) (layers F.Cu F.Paste F.Mask)
+      (net 54 "Net-(Q1-Pad2)"))
+    (pad 3 smd rect (at -1.25 0.95 180) (size 0.6 1.2) (layers F.Cu F.Paste F.Mask)
+      (net 1 GND))
+    (pad 4 smd rect (at 1.25 0.95 180) (size 0.6 1.2) (layers F.Cu F.Paste F.Mask)
+      (net 27 "Net-(IC3-Pad1)"))
+    (pad 5 smd rect (at 1.25 0 180) (size 0.6 1.2) (layers F.Cu F.Paste F.Mask)
+      (net 53 "Net-(Q1-Pad5)"))
+    (pad 6 smd rect (at 1.25 -0.95 180) (size 0.6 1.2) (layers F.Cu F.Paste F.Mask)
+      (net 34 "Net-(IC3-Pad3)"))
+    (model "${KIPRJMOD}/../FootPrints/3DModels/Sot23(6)/SOT23-6.stp"
+      (at (xyz 0 0 0))
+      (scale (xyz 1 1 1))

Commit message: Added changes
Parts:
- added R10: 10K, Encoder:R_0603_1608Metric_Pad1.05x0.95mm_HandSolder, F.Cu at (138.8, 90.5)
- added R12: 10K, Encoder:R_0603_1608Metric_Pad1.05x0.95mm_HandSolder, F.Cu at (137.2, 90.5)
- added R15: 10K, Encoder:R_0603_1608Metric_Pad1.05x0.95mm_HandSolder, F.Cu at (106.6, 124.3)
- added R16: 10K, Encoder:R_0603_1608Metric_Pad1.05x0.95mm_HandSolder, F.Cu at (106.6, 121.5)
- moved U4 7.04 mm to (126.8, 144.5)
- moved C18 6.36 mm to (121.3, 144.4), turned to 90 degrees
- moved C17 5.71 mm to (118.5, 144.4), turned to 90 degrees
- moved J2 1.32 mm to (128.2, 140.9)
- moved C15 1.09 mm to (131.6, 87.4), turned to 270 degrees
- moved C9 1.01 mm to (117.1, 99.4)
Connections:
- U1 pad 25: VCC -> Net-(R15-Pad2)
Routing:
- net Net-(R15-Pad2): track 0.00 -> 48.7 mm, vias 0 -> 4
- net VCC: track 115.0 -> 82.2 mm, vias 4 -> 0
- net /F1TX: track 34.1 -> 42.1 mm
- net /F1RX: track 35.3 -> 42.8 mm
- net +3V3: track 187.0 -> 190.8 mm, vias 0 -> 2
- net GND: track 95.4 -> 98.8 mm, vias 33 -> 34
- net /F1SCL: track 15.0 -> 14.2 mm

Commit message: Changes
Parts:
- moved J5 5.02 mm to (107.6, 131.2)
- moved S1 1.87 mm to (119.5, 127.8)
Routing:
- net VCC: track 82.2 -> 89.3 mm
- net /Batt+: track 25.9 -> 32.9 mm
- net GND: track 98.8 -> 95.1 mm
- net Net-(D1-Pad1): track 12.8 -> 10.6 mm
- net Net-(C11-Pad2): track 17.4 -> 15.6 mm

Commit message: New Changes
Parts:
- J1: footprint Encoder:PinSocket_1x07_P2.54mm_Vertical -> Encoder:PinHeader_1x07_P2.54mm_Vertical
- J5, J7: footprint Encoder:No3dmodelPinHeader_1x01_P2.54mm_Vertical -> Encoder:PinHeader_1x01_P2.54mm_Vertical_NO3D
- U1: footprint Encoder:QFP50P900X900X160-48N -> Encoder:LQFP-48_7x7mm_P0.5mm
