File: Mechatronics/Hardware/Electrical/BEncoder2Board/EncoderBoard2.kicad_pcb (KiCad board)
At the start: 2 copper layers, 37.8 x 63.5 mm, 94 parts, among them IC1 RN4020-V_RM120, IC1 TP4056, IC2 DW01+G, IC2 TP4056, IC3 DW01+G, J1 Conn_01x07_Male, J1 Conn_01x08_Male, J2 Conn_01x06_Male, J2 GNDPWR, J3 Barrel_Jack_Switch, J4 Barrel_Jack_Switch, J4 GNDPWR, J5 Batt+, J5 Conn_01x02_Male, J7 Batt-, Q1 DMosfet, Q2 Q_PMOS_GSD, Q3 Q_PMOS_GSD, U1 STM32F103C8T6, U1 STM32G431CBT6, U2 ITR1802, U3 ITR1802, U4 82402305, U4 RN4871, U5 82402305, U5 SSD1306OLED, U6 LTC3240, Y1 8Mhz

Commit message: Changes
Parts:
- moved S1 53.9 mm to (234.9, 135.4), turned to 270 degrees
- moved C17 52.9 mm to (240.0, 138.0), turned to 270 degrees
- moved C18 47.8 mm to (246.4, 135.4), turned to 270 degrees
- moved C16 45.2 mm to (240.0, 134.2), turned to 270 degrees
- moved IC1 41.8 mm to (217.2, 136.7)
- moved U6 40.7 mm to (243.8, 135.4)
- moved R10 40.1 mm to (243.8, 132.9)
- moved D1 38.9 mm to (229.9, 131.6), turned to 180 degrees
- moved J5 37.0 mm to (226.1, 136.7)
- moved R9 36.9 mm to (236.2, 132.9)
- moved IC2 35.6 mm to (217.2, 144.3)
- moved Q2 31.5 mm to (229.9, 139.2), turned to 270 degrees
- moved Q1 30.3 mm to (217.2, 148.1)
- moved R8 27.6 mm to (222.2, 139.2), turned to 270 degrees
- moved C15 26.0 mm to (219.7, 140.5), turned to 180 degrees
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Routing:
- net GND: track 83.2 -> 85.9 mm, vias 30 -> 32
- net Batt-: track 2.75 -> 0.00 mm, vias 2 -> 0

Commit message: Change s
Parts:
- moved J2 91.8 mm to (185.4, 101.1)
- moved R1 88.0 mm to (172.7, 110.0), turned to 90 degrees
- moved R2 84.9 mm to (172.7, 115.1), turned to 270 degrees
- moved U4 83.9 mm to (186.7, 92.3), turned to 0 degrees
- moved U2 83.2 mm to (176.5, 107.5), turned to 90 degrees
- moved Q3 78.4 mm to (174.0, 120.2), turned to 180 degrees
- moved U3 78.1 mm to (176.5, 114.9), turned to 90 degrees
- moved R3 76.0 mm to (181.6, 109.0), turned to 90 degrees
- moved R4 73.2 mm to (181.6, 112.7), turned to 90 degrees
- moved C11 73.1 mm to (195.6, 94.8), turned to 90 degrees
- moved C1 72.2 mm to (176.5, 125.3), turned to 90 degrees
- moved C9 72.0 mm to (184.8, 106.9), turned to 270 degrees
- moved C3 71.7 mm to (179.1, 120.2)
- moved R5 70.7 mm to (181.6, 116.4), turned to 270 degrees
- moved C8 70.4 mm to (191.8, 107.5), turned to 180 degrees
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Connections:
- C1 pad 1: Batt- -> GND
- C10 pad 2: Batt- -> GND
- C11 pad 2: Batt- -> GND
- C12 pad 2: Batt- -> GND
- C13 pad 2: Batt- -> GND
- C14 pad 2: Batt- -> GND
- C16 pad 1: Batt- -> GND
- C17 pad 2: Batt- -> GND
- C2 pad 1: Batt- -> GND
- C4 pad 2: Batt- -> GND
- C5 pad 2: Batt- -> GND
- C6 pad 2: Batt- -> GND
- C7 pad 2: Batt- -> GND
- C8 pad 2: Batt- -> GND
- C9 pad 1: Batt- -> GND
- IC1 pad 1: Batt- -> GND
- IC1 pad 3: Batt- -> GND
- J2 pad 3: Batt- -> GND
- J3 pad 2: Batt- -> GND
- J3 pad 3: Batt- -> GND
- J4 pad 1: Batt- -> GND
- Q1 pad 1: Batt- -> GND
- R1 pad 2: Batt- -> GND
- R2 pad 2: Batt- -> GND
- R5 pad 2: Batt- -> GND
- R6 pad 2: Batt- -> GND
- R7 pad 2: Batt- -> GND
- R9 pad 2: Batt- -> GND
- S1 pad 3: Batt- -> GND
- U1 pad 19: Batt- -> GND
- U1 pad 22: /BLERX -> Net-(U1-Pad22)
- U1 pad 23: Batt- -> GND
- U1 pad 25: /BLETX -> Net-(U1-Pad25)
- U1 pad 32: Net-(U1-Pad32) -> /BLETX
- U1 pad 35: Batt- -> GND
- U1 pad 43: /EncEnable -> /BLERX
- U1 pad 46: Net-(U1-Pad46) -> /EncEnable
- U1 pad 47: Batt- -> GND
- U2 pad 4: Batt- -> GND
- U3 pad 4: Batt- -> GND
- U4 pad 13: Batt- -> GND
- U4 pad 2: Batt- -> GND
- U5 pad 2: Batt- -> GND
- U6 pad 1: Batt- -> GND
- U6 pad 7: Batt- -> GND
Routing:
- net CHG: track 0.00 -> 55.2 mm
- net /BLERX: track 0.00 -> 51.0 mm
- net /Supply: track 0.00 -> 30.6 mm
- net +3V3: track 180.7 -> 206.2 mm
- net Batt-: track 0.00 -> 23.8 mm
- net /BLETX: track 0.00 -> 18.6 mm
- net Net-(D1-Pad1): track 10.6 -> 28.9 mm
- net /SWCLK: track 7.16 -> 25.2 mm
- net /2COS-: track 0.00 -> 17.8 mm
- net /LPTIM1_IN2: track 0.00 -> 15.4 mm
- net Net-(C1-Pad2): track 0.00 -> 15.2 mm
- net /SWDIO: track 3.12 -> 17.8 mm
- net GND: track 85.9 -> 100.4 mm, vias 32 -> 33
- net Batt+: track 0.00 -> 14.4 mm
- net /EncEnable: track 11.0 -> 24.3 mm
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
Commit message: Advances
Parts:
- removed the C1 at (115.2, 100.7)
- removed the C1 at (176.5, 125.3)
- removed the C10 at (127.6, 109.2)
- removed the C10 at (194.3, 98.6)
- removed the C11 at (128.4, 131.3)
- removed the C11 at (195.6, 94.8)
- removed the C12 at (131.8, 131.3)
- removed the C12 at (172.7, 141.8)
- removed the C13 at (113.1, 144.2)
- removed the C13 at (172.5, 138.6)
- removed the C14 at (130.6, 126.5)
- removed the C14 at (181.6, 146.9)
- removed the C15 at (131.6, 87.4)
- removed the C15 at (189.2, 137.3)
- removed the C16 at (120.1, 133.9)
- removed the C16 at (194.3, 135.4)
- removed the C17 at (118.5, 144.4)
- removed the C17 at (198.1, 135.4)
- removed the C18 at (121.3, 144.4)
- removed the C18 at (195.6, 129.1)
- removed the C2 at (114.8, 105.4)
- removed the C2 at (191.8, 125.3)
- removed the C3 at (115.2, 109.2)
- removed the C3 at (179.1, 120.2)
- removed the C4 at (115.2, 110.8)
- removed the C4 at (193.0, 121.5)
- removed the C5 at (127.5, 99.7)
- removed the C5 at (184.2, 118.9)
- removed the C6 at (130.6, 99.7)
- removed the C6 at (193.0, 105.0)
- removed the C7 at (108.6, 95.6)
- removed the C7 at (193.0, 102.4)
- removed the C8 at (108.9, 110.9)
- removed the C8 at (191.8, 107.5)
- removed the C9 at (117.1, 99.4)
- removed the C9 at (184.8, 106.9)
- removed the D1 at (114.3, 124.2)
- removed the D1 at (177.8, 132.9)
- removed the IC1 at (123.8, 90.6)
- removed the IC1 at (180.3, 140.5)
- removed the IC2 at (115.6, 137.2)
- removed the IC2 at (188.0, 140.5)
- removed IC3: DW01+G, Encoder:Sot-23(6)
- removed the J1 at (134.4, 104.9)
- removed the J1 at (198.1, 121.5)
- removed the J2 at (128.2, 140.9)
- removed the J2 at (185.4, 101.1)
- removed the J4 at (135.0, 139.2)
- removed the J4 at (174.0, 135.4)
- removed the J5 at (107.6, 131.2)
- removed the J5 at (185.4, 136.1)
- removed J7: Batt-, Encoder:No3dmodelPinHeader_1x01_P2.54mm_Vertical
- removed the Q1 at (124.5, 137.1)
- removed the Q1 at (188.0, 145.6)
- removed the Q2 at (112.6, 127.7)
- removed the Q2 at (181.6, 134.2)
- removed the R10 at (138.8, 90.5)
- removed the R10 at (193.0, 131.6)
- removed the R5 at (120.4, 110.6)
- removed the R5 at (181.6, 116.4)
- removed the R6 at (110.1, 127.7)
- removed the R6 at (179.1, 145.6)
- removed the R7 at (127.5, 127.8)
- removed the R7 at (185.4, 142.4)
- removed the R8 at (114.9, 142.6)
- removed the R8 at (189.2, 135.4)
- removed the R9 at (121.6, 141.4)
- removed the R9 at (176.5, 139.2)
- removed the S1 at (119.5, 127.8)
- removed the S1 at (193.1, 138.0)
- removed the U1 at (189.2, 113.8)
- removed the U1 at (122.8, 104.7)
- removed the U4 at (126.8, 144.5)
- removed the U4 at (186.7, 92.3)
- removed the U5 at (111.2, 87.8)
- removed the U5 at (175.3, 145.6)
- removed the U6 at (129.6, 129.0)
- removed the U6 at (195.6, 131.6)
- removed the Y1 at (110.1, 100.7)
- removed the Y1 at (186.7, 124.0)
- added C1: 12pF, Encoder:C_0603_1608Metric_Pad1.05x0.95mm_HandSolder, F.Cu at (110.5, 122.7)
- added C10: 1uF, Encoder:C_0603_1608Metric_Pad1.05x0.95mm_HandSolder, F.Cu at (128.0, 95.2)
- added C11: 10uF, Encoder:C_0603_1608Metric_Pad1.05x0.95mm_HandSolder, F.Cu at (128.0, 91.7)
- added C12: 1uF, Encoder:C_0603_1608Metric_Pad1.05x0.95mm_HandSolder, F.Cu at (110.7, 137.3)
- added C13: 1uF, Encoder:C_0603_1608Metric_Pad1.05x0.95mm_HandSolder, F.Cu at (110.5, 134.2)
- added C14: 10uF, Encoder:C_0603_1608Metric_Pad1.05x0.95mm_HandSolder, F.Cu at (120.0, 141.7)
- added C15: .1uF, Encoder:C_0603_1608Metric_Pad1.05x0.95mm_HandSolder, F.Cu at (127.3, 132.9)
- added C16: 1uF, Encoder:C_0603_1608Metric_Pad1.05x0.95mm_HandSolder, F.Cu at (132.2, 133.1)
- added C17: 4.7uF, Encoder:C_0603_1608Metric_Pad1.05x0.95mm_HandSolder, F.Cu at (136.0, 133.1)
- added C18: 1uF, Encoder:C_0603_1608Metric_Pad1.05x0.95mm_HandSolder, F.Cu at (133.5, 126.8)
- added C19: 3.2uF, Encoder:C_0603_1608Metric_Pad1.05x0.95mm_HandSolder, F.Cu at (132.8, 118.9)
- added C2: 12pF, Encoder:C_0603_1608Metric_Pad1.05x0.95mm_HandSolder, F.Cu at (125.7, 122.7)
- added C20: 3.2uF, Encoder:C_0603_1608Metric_Pad1.05x0.95mm_HandSolder, F.Cu at (134.9, 114.4)
- added C21: 3.2uF, Encoder:C_0603_1608Metric_Pad1.05x0.95mm_HandSolder, F.Cu at (133.0, 107.5)
- added C22: 3.2uF, Encoder:C_0603_1608Metric_Pad1.05x0.95mm_HandSolder, F.Cu at (135.0, 105.1)
- added C23: 3.2uF, Encoder:C_0603_1608Metric_Pad1.05x0.95mm_HandSolder, F.Cu at (133.3, 98.0)
- added C24: 3.2uF, Encoder:C_0603_1608Metric_Pad1.05x0.95mm_HandSolder, F.Cu at (136.3, 98.0)
- added C25: 3.2uF, Encoder:C_0603_1608Metric_Pad1.05x0.95mm_HandSolder, F.Cu at (134.4, 91.1)
- added C26: 3.2uF, Encoder:C_0603_1608Metric_Pad1.05x0.95mm_HandSolder, F.Cu at (137.4, 91.1)
- added C3: 4.7uF, Encoder:C_0603_1608Metric_Pad1.05x0.95mm_HandSolder, F.Cu at (113.0, 117.7)
- added C4: 100nF, Encoder:C_0603_1608Metric_Pad1.05x0.95mm_HandSolder, F.Cu at (127.0, 120.2)
- added C5: 100nF, Encoder:C_0603_1608Metric_Pad1.05x0.95mm_HandSolder, F.Cu at (118.1, 116.4)
- added C6: 1uF, Encoder:C_0603_1608Metric_Pad1.05x0.95mm_HandSolder, F.Cu at (127.3, 102.3)
- added C7: 10nF, Encoder:C_0603_1608Metric_Pad1.05x0.95mm_HandSolder, F.Cu at (127.3, 100.0)
- added C8: 100nF, Encoder:C_0603_1608Metric_Pad1.05x0.95mm_HandSolder, F.Cu at (127.0, 105.0)
- added C9: 100nF, Encoder:C_0603_1608Metric_Pad1.05x0.95mm_HandSolder, F.Cu at (118.7, 104.3)
- added D1: D, Encoder:D_SMA, F.Cu at (115.8, 128.4)
- added IC1: TP4056, Encoder:Sop(8), F.Cu at (118.4, 136.1)
- added IC2: DW01+G, Encoder:Sot-23(6), F.Cu at (126.0, 136.0)
- added J1: Conn_01x08_Male, Encoder:PinHeader_1x08_P2.54mm_Vertical, F.Cu at (138.2, 122.7)
- added J2: Conn_01x06_Male, Encoder:PinHeader_1x06_P2.54mm_Vertical, F.Cu at (123.3, 98.7)
- added J4: GNDPWR, Encoder:PinHeader_1x01_P2.54mm_Vertical, F.Cu at (112.0, 131.0)
- added J5: Conn_01x02_Male, Encoder:PinHeader_1x02_P2.54mm_Vertical, F.Cu at (123.4, 131.6)
- added Q1: DMosfet, Encoder:Sot-23(6), F.Cu at (126.0, 141.1)
- added Q2: Q_PMOS_GSD, Encoder:SOT-23, F.Cu at (119.6, 129.7)
- added R10: 10K, Encoder:R_0603_1608Metric_Pad1.05x0.95mm_HandSolder, F.Cu at (130.9, 129.3)
- added R17: 100, Encoder:R_0603_1608Metric_Pad1.05x0.95mm_HandSolder, F.Cu at (134.4, 94.5)
- added R18: 100, Encoder:R_0603_1608Metric_Pad1.05x0.95mm_HandSolder, F.Cu at (137.4, 94.5)
- added R5: 10K, Encoder:R_0603_1608Metric_Pad1.05x0.95mm_HandSolder, F.Cu at (115.6, 113.8)
- added R6: 1.2K, Encoder:R_0603_1608Metric_Pad1.05x0.95mm_HandSolder, F.Cu at (117.1, 141.1)
- added R7: 1K, Encoder:R_0603_1608Metric_Pad1.05x0.95mm_HandSolder, F.Cu at (123.4, 138.0)
- added R8: 100, Encoder:R_0603_1608Metric_Pad1.05x0.95mm_HandSolder, F.Cu at (127.3, 131.0)
- added R9: 10K, Encoder:R_0603_1608Metric_Pad1.05x0.95mm_HandSolder, F.Cu at (114.6, 134.8)
- added S1: EG1218, Encoder:Switch_Slide_11.6x4mm_EG1218, F.Cu at (131.2, 135.4)
- added U1: STM32G431CBT6, Encoder:LQFP-48_7x7mm_P0.5mm, F.Cu at (123.2, 111.3)
- added U4: RN4871, Encoder:Bluetooth_Module_RN4871, F.Cu at (120.7, 89.7)
- added U5: 82402305, Encoder:Sot-23(6), F.Cu at (113.3, 141.1)
- added U6: LTC3240, Encoder:DFN-6_DC, F.Cu at (133.5, 129.3)
- added Y1: 8Mhz, Encoder:Crystal_HC49-U_Vertical, F.Cu at (120.7, 121.5)
- R12, R13, R14, R15, R16: value 10K -> 100
- moved R3 66.1 mm to (115.6, 106.5)
- moved R4 66.1 mm to (115.6, 110.2)
- moved Q3 66.1 mm to (108.0, 117.7), turned to 90 degrees
- moved R1 65.1 mm to (107.7, 107.2)
- moved R2 65.1 mm to (107.7, 112.3)
- moved U2 65.1 mm to (111.5, 104.7)
- moved U3 65.1 mm to (111.5, 112.1)
- moved J3 61.0 mm to (134.6, 138.9)
- moved R16 35.8 mm to (136.3, 101.4), turned to 270 degrees
- moved R15 35.2 mm to (133.3, 101.4), turned to 270 degrees
- moved R12 27.4 mm to (134.9, 117.8)
- moved R14 24.6 mm to (135.0, 108.5), turned to 270 degrees
- moved R13 22.8 mm to (133.0, 110.9), turned to 270 degrees
- moved R11 17.8 mm to (132.8, 122.4), turned to 270 degrees
Connections:
- R11 pad 1: /Batt+ -> /1SIN+
- R12 pad 1: +3V3 -> /1SIN-
- R12 pad 2: /F1RX -> Net-(J1-Pad2)
- R13 pad 1: /Batt+ -> /1COS+
- R13 pad 2: Net-(R13-Pad2) -> Net-(J1-Pad3)
- R14 pad 1: Net-(R13-Pad2) -> /1COS-
- R14 pad 2: GND -> Net-(J1-Pad4)
- R15 pad 1: VCC -> /2COS-
- R15 pad 2: Net-(R15-Pad2) -> Net-(J1-Pad5)
- R16 pad 1: Net-(R15-Pad2) -> /2SIN+
- R16 pad 2: GND -> Net-(J1-Pad6)
Routing:
- net Batt+: track 14.4 -> 153.1 mm
- net GND: track 100.4 -> 1.41 mm, vias 33 -> 1
- net VCC: track 89.3 -> 0.00 mm
- net CHG: track 55.2 -> 123.8 mm
- net Net-(R15-Pad2): track 48.7 -> 0.00 mm, vias 4 -> 0
- net /F1RX: track 39.3 -> 0.00 mm
- net /Batt+: track 32.9 -> 0.00 mm
- net /F1TX: track 27.1 -> 0.00 mm
- net /2SIN+: track 7.44 -> 27.5 mm
- net /2COS+: track 10.3 -> 29.8 mm
- net /1COS-: track 0.00 -> 19.1 mm
- net /2SIN-: track 9.27 -> 25.5 mm
- net Net-(IC3-Pad1): track 16.1 -> 0.00 mm
- net Net-(J1-Pad7): track 0.00 -> 15.0 mm
- net Net-(R13-Pad2): track 15.0 -> 0.00 mm
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Other:
- net class Default: clearance 0.1016 -> 0.127; trace_width 0.1016 -> 0.127
- rule trace_clearance: 0.1016 -> 0.127

Commit message: Changes
Parts:
- moved C14 4.51 mm to (116.2, 144.1), turned to 180 degrees
- moved C5 2.54 mm to (116.1, 117.9), turned to 0 degrees
- moved J4 2.39 mm to (109.9, 132.0)
- moved D1 1.80 mm to (114.0, 128.7)
- moved Q2 1.77 mm to (118.0, 130.4)
- moved R9 1.55 mm to (113.0, 135.1)
- moved R8 1.45 mm to (126.1, 130.1)
- moved C4 1.30 mm to (125.7, 120.4)
- moved C15 1.25 mm to (126.1, 132.4)
- moved C13 1.18 mm to (109.7, 135.1)
- moved C12 1.05 mm to (109.7, 137.6)
- moved J3 0.92 mm to (133.7, 139.1)
- moved U5 0.92 mm to (112.4, 141.4)
- moved C2 0.92 mm to (124.8, 123.0)
- moved C22 0.92 mm to (134.1, 105.3)
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Connections:
- U1 pad 26: Net-(U1-Pad26) -> CHG
- U1 pad 27: CHG -> Net-(U1-Pad27)
Routing:
- net GND: track 1.41 -> 63.6 mm, vias 1 -> 33
- net CHG: track 123.8 -> 135.2 mm
- net Net-(C4-Pad1): track 0.00 -> 6.12 mm
- net Batt-: track 23.8 -> 18.0 mm
- net Net-(IC2-Pad1): track 6.71 -> 10.7 mm
- net Net-(IC2-Pad3): track 0.30 -> 4.13 mm
- net /EncEnable: track 12.0 -> 14.9 mm
- net Net-(C15-Pad1): track 5.01 -> 6.91 mm
- net Net-(D1-Pad1): track 24.9 -> 26.8 mm
- net Batt+: track 153.1 -> 154.7 mm
- net /LPTIM1_IN1: track 9.61 -> 11.0 mm
- net +3V3: track 192.3 -> 193.2 mm
- net Net-(J1-Pad1): track 5.92 -> 5.22 mm
Other:
- board size 37.8 x 63.5 mm -> 37.8 x 59.2 mm

Commit message: Changes
Routing:
- net GND: track 63.6 -> 70.4 mm, vias 33 -> 37
- net +3V3: track 193.2 -> 193.9 mm
Other:
- rule trace_min: 0.0889 -> 0.127

Commit message: Finished PCB
Parts:
- added R19: 10K, Encoder:R_0603_1608Metric_Pad1.05x0.95mm_HandSolder, F.Cu at (106.2, 144.6)
- added R20: 10K, Encoder:R_0603_1608Metric_Pad1.05x0.95mm_HandSolder, F.Cu at (108.6, 144.6)
- S1: value EG1218 -> EG1218(+3.3v); footprint Encoder:Switch_Slide_11.6x4mm_EG1218 -> Encoder:PinHeader_1x04_P2.54mm_Vertical
- moved R1 2.80 mm to (106.7, 104.7)
- moved R11 2.17 mm to (131.7, 120.4)
- moved C19 2.17 mm to (131.7, 117.0)
- moved C17 1.91 mm to (135.3, 131.5)
- moved C16 1.91 mm to (131.4, 131.5)
- moved R3 1.78 mm to (114.7, 105.0)
- moved R10 1.59 mm to (130.8, 128.2)
- moved C18 1.27 mm to (133.3, 126.0)
- moved U6 1.27 mm to (133.3, 128.6)
- moved S1 0.96 mm to (131.1, 135.1), turned to 90 degrees
- moved U5 0.89 mm to (111.5, 141.4)
- moved R6 0.80 mm to (115.4, 141.1)
- moved C14 0.77 mm to (115.4, 144.2)
- moved R2 0.40 mm to (106.7, 112.2), turned to 90 degrees
- moved U3 0.13 mm to (110.6, 112.4)
Connections:
- net CHG renamed VCC
- U1 pad 28: Batt+ -> Net-(R19-Pad2)
Routing:
- net Net-(R19-Pad2): track 0.00 -> 125.5 mm
- net Batt+: track 154.7 -> 38.0 mm
- net GND: track 70.4 -> 77.2 mm, vias 37 -> 38
- net +3V3: track 193.9 -> 200.0 mm
- net VCC: track 135.2 -> 140.3 mm
- net Net-(Q3-Pad3): track 21.8 -> 24.1 mm
- net Net-(R1-Pad1): track 6.68 -> 4.44 mm
- net /SWDIO: track 12.2 -> 14.2 mm
- net /SWCLK: track 14.5 -> 16.2 mm
- net Net-(R2-Pad1): track 3.19 -> 4.53 mm
- net Net-(C16-Pad2): track 9.67 -> 10.8 mm
- net Net-(J1-Pad1): track 5.22 -> 6.28 mm
- net /LPTIM1_IN2: track 14.9 -> 15.9 mm
- net (no net): vias 1 -> 0
Other:
- board text added: "+"
- board text added: "-"
- board text added: "1C+"
- board text added: "1C-"
- board text added: "1S+"
- board text added: "1S-"
- board text added: "2C+"
- board text added: "2C-"
- board text added: "2S+"
- board text added: "2S-"
- board text added: "3.3V"
- board text added: "<>"
- board text added: "Boot0"
- board text added: "CLK"
- board text added: "D+"
- board text added: "D-"
- board text added: "DIO"
- board text added: "E+"
- board text added: "E-"
- board text added: "GND"
- board text added: "SCL"
- board text added: "SDA"
- board text added: "VCC"

Commit message: Changes
Parts:
- added J6: Conn_01x04_Male, Encoder:PinHeader_2x02_P2.54mm_Vertical, F.Cu at (108.6, 91.6)
Routing:
- net +3V3: track 200.0 -> 207.2 mm
Other:
- board text added: "GNDPWR"

Commit message: Changes
Parts:
- moved C5 0.69 mm to (116.8, 117.9)
Connections:
- C3 pad 2: /Supply -> GND
- C5 pad 1: /Supply -> +3V3
- C8 pad 1: /Supply -> +3V3
- C9 pad 2: /Supply -> +3V3
- U1 pad 24: /Supply -> +3V3
- U1 pad 36: /Supply -> +3V3
- U1 pad 48: /Supply -> +3V3
Routing:
- net +3V3: track 207.2 -> 241.4 mm
- net /Supply: track 31.2 -> 0.00 mm
- net GND: track 77.1 -> 78.4 mm, vias 38 -> 39
