File: Mechatronics/Hardware/Electrical/BEncoder2Board/EncoderBoard2.kicad_pcb (KiCad board)
At the start: 2 copper layers, 37.8 x 59.2 mm, 66 parts, among them IC1 TP4056, IC2 DW01+G, J1 Conn_01x08_Male, J2 Conn_01x06_Male, J3 Barrel_Jack_Switch, J4 GNDPWR, J5 Conn_01x02_Male, J6 Conn_01x04_Male, Q1 DMosfet, Q2 Q_PMOS_GSD, Q3 Q_PMOS_GSD, U1 STM32G431CBT6, U2 ITR1802, U3 ITR1802, U4 RN4871, U5 82402305, U6 LTC3240, Y1 8Mhz

Commit message: Final PCB
Parts:
- J2: value Conn_01x06_Male -> Conn_01x07_Male; footprint Encoder:PinHeader_1x06_P2.54mm_Vertical -> Encoder:PinHeader_1x07_P2.54mm_Vertical
- moved C6 1.15 mm to (127.5, 102.7)
- moved C7 1.15 mm to (127.5, 100.4)
- moved C9 0.92 mm to (118.7, 104.3)
- moved J2 0.89 mm to (123.3, 99.0)
Routing:
- net +3V3: track 241.4 -> 246.3 mm
- net /SWDIO: track 14.2 -> 12.4 mm
- net /BLERX: track 52.7 -> 53.7 mm
- net /SWCLK: track 16.2 -> 15.4 mm
- net VCC: track 140.3 -> 139.7 mm
