File: Mechatronics/Hardware/Electrical/BEncoder2Board/EncoderBoard2.sch (KiCad schematic (older format))
At the start: 24 parts, among them J1 Conn_01x08_Male, J2 Conn_01x08_Male, Q3 Q_PMOS_GSD, U1 STM32G431CBT6, U2 ITR1802, U3 ITR1802, U4 RN4871, Y1 8Mhz

Commit message: New Changes
Parts:
- removed J2: Conn_01x08_Male, symbol Connector:Conn_01x08_Male
- added J2: Conn_01x06_Male, Encoder:PinHeader_1x06_P2.54mm_Vertical, symbol Connector:Conn_01x06_Male
- C10, C11, C3, C4, C5, C6, C7, C8, C9: footprint (none) -> Encoder:C_0603_1608Metric_Pad1.05x0.95mm_HandSolder
- J1: footprint (none) -> Encoder:PinHeader_1x08_P2.54mm_Vertical
- U1: footprint (none) -> Encoder:LQFP-48_7x7mm_P0.5mm
- U4: footprint (none) -> Encoder:Bluetooth_Module_RN4871
Connections:
- net labels added: CHG
- wire segments 101 -> 100
- no-connect marks 25 -> 24
Other:
- moved on the sheet: C6
Changed lines of the file:
@@
 F 0 "U4" H 7550 6215 50  0000 C CNN
 F 1 "RN4871" H 7550 6124 50  0000 C CNN
-F 2 "" H 7450 5550 50  0001 C CNN
+F 2 "Encoder:Bluetooth_Module_RN4871" H 7450 5550 50  0001 C CNN
 F 3 "" H 7450 5550 50  0001 C CNN
 	1    7500 5450
@@
 F 0 "C8" H 5115 6996 50  0000 L CNN
 F 1 "100nF" H 5115 6905 50  0000 L CNN
-F 2 "" H 5038 6800 50  0001 C CNN
+F 2 "Encoder:C_0603_1608Metric_Pad1.05x0.95mm_HandSolder" H 5038 6800 50  0001 C CNN
 F 3 "~" H 5000 6950 50  0001 C CNN
 	1    5000 6950
@@
 F 0 "C9" V 5498 4600 50  0000 C CNN
 F 1 "100nF" V 5589 4600 50  0000 C CNN
-F 2 "" H 5788 4450 50  0001 C CNN
+F 2 "Encoder:C_0603_1608Metric_Pad1.05x0.95mm_HandSolder" H 5788 4450 50  0001 C CNN
 F 3 "~" H 5750 4600 50  0001 C CNN
 	1    5750 4600
@@
 F 0 "C3" H 2565 4046 50  0000 L CNN
 F 1 "4.7uF" H 2565 3955 50  0000 L CNN
-F 2 "" H 2488 3850 50  0001 C CNN
+F 2 "Encoder:C_0603_1608Metric_Pad1.05x0.95mm_HandSolder" H 2488 3850 50  0001 C CNN
 F 3 "~" H 2450 4000 50  0001 C CNN
 	1    2450 4000
@@
 $EndComp
 Wire Wire Line
-	2450 4150 2450 4550
+	2450 4150 2450 4500
 Text Label 2450 4150 3    50   ~ 0
 Supply
@@
 F 0 "C5" V 2848 3950 50  0000 C CNN
 F 1 "100nF" V 2939 3950 50  0000 C CNN
-F 2 "" H 3138 3800 50  0001 C CNN
+F 2 "Encoder:C_0603_1608Metric_Pad1.05x0.95mm_HandSolder" H 3138 3800 50  0001 C CNN
 F 3 "~" H 3100 3950 50  0001 C CNN
 	1    3100 3950
 	0    1    1    0
 $EndComp
-$Comp
-L Encoder:STM32G431CBT6 U1
-U 1 1 5EF8C6BF
-P 4150 5450
-F 0 "U1" H 4100 5600 50  0000 L CNN
-F 1 "STM32G431CBT6" H 3850 5400 50  0000 L CNN
-F 2 "" H 3850 5600 50  0001 C CNN
-F 3 "" H 3850 5600 50  0001 C CNN
-	1    4150 5450
-	1    0    0    -1
-$EndComp
 Wire Wire Line
 	3350 3500 3350 3950
@@
 U 1 1 5F05A8A9
 P 4550 7400
-F 0 "C7" H 4300 7450 50  0000 L CNN
-F 1 "10nF" H 4250 7300 50  0000 L CNN
-F 2 "" H 4588 7250 50  0001 C CNN
+F 0 "C7" H 4400 7500 50  0000 L CNN
+F 1 "10nF" H 4350 7300 50  0000 L CNN
+F 2 "Encoder:C_0603_1608Metric_Pad1.05x0.95mm_HandSolder" H 4588 7250 50  0001 C CNN
 F 3 "~" H 4550 7400 50  0001 C CNN
 	1    4550 7400
@@
 $EndComp
 $Comp
-L Device:C C6
-U 1 1 5F05B729
-P 4050 7400
-F 0 "C6" H 3850 7450 50  0000 L CNN
-F 1 "1uF" H 3850 7300 50  0000 L CNN
-F 2 "" H 4088 7250 50  0001 C CNN
-F 3 "~" H 4050 7400 50  0001 C CNN
-	1    4050 7400
-	1    0    0    -1
-$EndComp
-Wire Wire Line
-	4550 6650 4550 7250
-$Comp
 L power:+3.3V #PWR0108
 U 1 1 5F07D03B
-P 4050 7250
-F 0 "#PWR0108" H 4050 7100 50  0001 C CNN
-F 1 "+3.3V" V 4065 7378 50  0000 L CNN
-F 2 "" H 4050 7250 50  0001 C CNN
-F 3 "" H 4050 7250 50  0001 C CNN
-	1    4050 7250
-	0    -1   -1   0
+P 4250 7250
+F 0 "#PWR0108" H 4250 7100 50  0001 C CNN
+F 1 "+3.3V" H 4265 7378 50  0000 L CNN
+F 2 "" H 4250 7250 50  0001 C CNN
+F 3 "" H 4250 7250 50  0001 C CNN
+	1    4250 7250
+	1    0    0    -1
 $EndComp
 $Comp
@@
 L power:GND #PWR0114
 U 1 1 5F07F709
-P 4050 7550
-F 0 "#PWR0114" H 4050 7300 50  0001 C CNN
-F 1 "GND" H 4055 7377 50  0000 C CNN
-F 2 "" H 4050 7550 50  0001 C CNN
-F 3 "" H 4050 7550 50  0001 C CNN
-	1    4050 7550
+P 4250 7550
+F 0 "#PWR0114" H 4250 7300 50  0001 C CNN
+F 1 "GND" H 4255 7377 50  0000 C CNN
+F 2 "" H 4250 7550 50  0001 C CNN
+F 3 "" H 4250 7550 50  0001 C CNN
+	1    4250 7550
 	1    0    0    -1
 $EndComp
@@
 F 0 "C4" V 2500 5450 50  0000 C CNN
 F 1 "100nF" V 2650 5300 50  0000 C CNN
-F 2 "" H 2738 5350 50  0001 C CNN
+F 2 "Encoder:C_0603_1608Metric_Pad1.05x0.95mm_HandSolder" H 2738 5350 50  0001 C CNN
 F 3 "~" H 2700 5500 50  0001 C CNN
 	1    2700 5500
@@
 Wire Wire Line
 	3800 4100 3800 3850
-Wire Wire Line
-	3350 6650 3350 7050
-Wire Wire Line
-	3500 6650 3500 7050
-Wire Wire Line
-	3650 6650 3650 7050
-Wire Wire Line
-	4100 6650 4100 7050
-Wire Wire Line
-	3800 6650 3800 7050
-Text Label 3800 6950 1    50   ~ 0
-Batt+
 Text Label 3500 6950 1    50   ~ 0
 2SIN+
@@
 F 0 "C10" H 8265 6196 50  0000 L CNN
 F 1 "1uF" H 8265 6105 50  0000 L CNN
-F 2 "" H 8188 6000 50  0001 C CNN
+F 2 "Encoder:C_0603_1608Metric_Pad1.05x0.95mm_HandSolder" H 8188 6000 50  0001 C CNN
 F 3 "~" H 8150 6150 50  0001 C CNN
 	1    8150 6150
@@
 F 0 "C11" H 8765 5396 50  0000 L CNN
 F 1 "10uF" H 8765 5305 50  0000 L CNN
-F 2 "" H 8688 5200 50  0001 C CNN
+F 2 "Encoder:C_0603_1608Metric_Pad1.05x0.95mm_HandSolder" H 8688 5200 50  0001 C CNN
 F 3 "~" H 8650 5350 50  0001 C CNN
 	1    8650 5350
@@
 Wire Wire Line
 	5450 6250 6250 6250
-Wire Wire Line
-	4700 6650 4700 7600
 Text Label 4700 7050 1    50   ~ 0
 USART3TX
@@
 I2C2SDA
 Wire Wire Line
-	4550 7250 4050 7250
+	4550 7250 4250 7250
 Connection ~ 4550 7250
-Connection ~ 4050 7250
 $Sheet
 S 7900 1500 700  350
@@
 F 0 "J1" H 2000 6850 50  0000 C CNN
 F 1 "Conn_01x08_Male" H 2350 7300 50  0000 C CNN
-F 2 "" H 2100 6850 50  0001 C CNN
+F 2 "Encoder:PinHeader_1x08_P2.54mm_Vertical" H 2100 6850 50  0001 C CNN
 F 3 "~" H 2100 6850 50  0001 C CNN
 	1    2100 6850
@@
 Text Label 2350 6850 0    50   ~ 0
 1COS-
+Text Label 2600 7250 2    50   ~ 0
+2COS-
 Text Label 2600 6950 2    50   ~ 0
-2COS-
+2SIN+
 Text Label 2600 7050 2    50   ~ 0
-2SIN+
+2SIN-
 Text Label 2600 7150 2    50   ~ 0
-2SIN-
-Text Label 2600 7250 2    50   ~ 0
 2COS+
 $Comp
@@
 Wire Wire Line
 	6850 3850 6500 3850
-Wire Wire Line
-	6850 3950 6500 3950
-Wire Wire Line
-	6850 4050 6500 4050
-Text Label 6850 4050 2    50   ~ 0
-BLERX
-Text Label 6850 3950 2    50   ~ 0
-BLETX
 Text Label 6850 3850 2    50   ~ 0
 OLEDSDA
@@
 Wire Wire Line
 	6400 3650 6850 3650
-$Comp
-L Connector:Conn_01x08_Male J2
-U 1 1 5F23D818
-P 7050 3750
-F 0 "J2" H 7022 3632 50  0000 R CNN
-F 1 "Conn_01x08_Male" H 7022 3723 50  0000 R CNN
-F 2 "" H 7050 3750 50  0001 C CNN
-F 3 "~" H 7050 3750 50  0001 C CNN
-	1    7050 3750
-	-1   0    0    1
-$EndComp
 Text Label 6850 3450 2    50   ~ 0
 SWDIO
@@
 OLEDSDA
 NoConn ~ 3650 4100
-NoConn ~ 4100 4100
 NoConn ~ 4400 4100
 NoConn ~ 2850 4750
 NoConn ~ 2850 4900
-NoConn ~ 2850 5050
 NoConn ~ 2850 6250
-NoConn ~ 3950 6650
 NoConn ~ 4400 6650
 NoConn ~ 5450 6100
@@
 NoConn ~ 5450 4900
 NoConn ~ 7800 5900
-$Comp
-L power:PWR_FLAG #FLG0102
-U 1 1 5F292D49
-P 2450 3900
-F 0 "#FLG0102" H 2450 3975 50  0001 C CNN
-F 1 "PWR_FLAG" V 2450 4027 50  0000 L CNN
-F 2 "" H 2450 3900 50  0001 C CNN
-F 3 "~" H 2450 3900 50  0001 C CNN
-	1    2450 3900
-	0    -1   -1   0
-$EndComp
 Text Label 4250 3500 1    50   ~ 0
 SIGA
+$Comp
+L Connector:Conn_01x06_Male J2
+U 1 1 5EFD316D
+P 7050 3650
+F 0 "J2" H 7022 3532 50  0000 R CNN
+F 1 "Conn_01x06_Male" H 7022 3623 50  0000 R CNN
+F 2 "Encoder:PinHeader_1x06_P2.54mm_Vertical" H 7050 3650 50  0001 C CNN
+F 3 "~" H 7050 3650 50  0001 C CNN
+	1    7050 3650
+	-1   0    0    1
+$EndComp
+Wire Wire Line
+	4100 4100 4100 3300
+Text Label 4100 3650 3    50   ~ 0
+EncEnable
+$Comp
+L power:PWR_FLAG #FLG0102
+U 1 1 5EFDA81C
+P 2450 4500
+F 0 "#FLG0102" H 2450 4575 50  0001 C CNN
+F 1 "PWR_FLAG" V 2450 4627 50  0000 L CNN
+F 2 "" H 2450 4500 50  0001 C CNN
+F 3 "~" H 2450 4500 50  0001 C CNN
+	1    2450 4500
+	0    -1   -1   0
+$EndComp
+Connection ~ 2450 4500
+Wire Wire Line
+	2450 4500 2450 4550
+Text GLabel 3800 6650 3    50   Input ~ 0
+Batt+
+Connection ~ 4250 7250
+$Comp
+L Device:C C6
+U 1 1 5F05B729
+P 4250 7400
+F 0 "C6" H 4050 7450 50  0000 L CNN
+F 1 "1uF" H 4050 7300 50  0000 L CNN
+F 2 "Encoder:C_0603_1608Metric_Pad1.05x0.95mm_HandSolder" H 4288 7250 50  0001 C CNN
+F 3 "~" H 4250 7400 50  0001 C CNN
+	1    4250 7400
+	1    0    0    -1
+$EndComp
+Text GLabel 3950 6650 3    50   Input ~ 0
+CHG
+NoConn ~ 2850 4600
+Wire Wire Line
+	3350 6650 3350 7050
+Wire Wire Line
+	3500 6650 3500 7050
+Wire Wire Line
+	3650 6650 3650 7050
+Wire Wire Line
+	4100 6650 4100 7050
+Wire Wire Line
+	4550 6650 4550 7250
+Wire Wire Line
+	4700 6650 4700 7600
+$Comp
+L Encoder:STM32G431CBT6 U1
+U 1 1 5EF8C6BF
+P 4150 5450
+F 0 "U1" H 4100 5600 50  0000 L CNN
+F 1 "STM32G431CBT6" H 3850 5400 50  0000 L CNN
+F 2 "Encoder:LQFP-48_7x7mm_P0.5mm" H 3850 5600 50  0001 C CNN
+F 3 "" H 3850 5600 50  0001 C CNN
+	1    4150 5450
+	1    0    0    -1
+$EndComp
+NoConn ~ 2850 5050
 $EndSCHEMATC

Commit message: Additions
Parts:
- U2, U3: footprint Encoder:OptointerrupterConnector -> Encoder:OptointerrupterSmall
Changed lines of the file:
@@
 F 0 "U2" H 3250 2125 50  0000 C CNN
 F 1 "ITR1802" H 3250 2034 50  0000 C CNN
-F 2 "Encoder:OptointerrupterConnector" H 3250 1800 50  0001 C CNN
+F 2 "Encoder:OptointerrupterSmall" H 3250 1800 50  0001 C CNN
 F 3 "" H 3250 1800 50  0001 C CNN
 	1    3250 1800
@@
 F 0 "U3" H 3250 3025 50  0000 C CNN
 F 1 "ITR1802" H 3250 2934 50  0000 C CNN
-F 2 "Encoder:OptointerrupterConnector" H 3250 2700 50  0001 C CNN
+F 2 "Encoder:OptointerrupterSmall" H 3250 2700 50  0001 C CNN
 F 3 "" H 3250 2700 50  0001 C CNN
 	1    3250 2700

Commit message: Change s
Connections:
- net labels added: USART1RX, USART1TX
- net labels removed: USART3RX, USART3TX
- wire segments 100 -> 99
Other:
- moved on the sheet: R5
Changed lines of the file:
@@
 L power:GND #PWR0120
 U 1 1 5F070E6F
-P 3650 3550
-F 0 "#PWR0120" H 3650 3300 50  0001 C CNN
-F 1 "GND" H 3655 3377 50  0000 C CNN
-F 2 "" H 3650 3550 50  0001 C CNN
-F 3 "" H 3650 3550 50  0001 C CNN
-	1    3650 3550
+P 3800 3350
+F 0 "#PWR0120" H 3800 3100 50  0001 C CNN
+F 1 "GND" H 3805 3177 50  0000 C CNN
+F 2 "" H 3800 3350 50  0001 C CNN
+F 3 "" H 3800 3350 50  0001 C CNN
+	1    3800 3350
 	-1   0    0    1
 $EndComp
@@
 L Device:R R5
 U 1 1 5F070E68
-P 3650 3700
-F 0 "R5" H 3720 3746 50  0000 L CNN
-F 1 "10K" H 3720 3655 50  0000 L CNN
-F 2 "Encoder:R_0603_1608Metric_Pad1.05x0.95mm_HandSolder" V 3580 3700 50  0001 C CNN
-F 3 "~" H 3650 3700 50  0001 C CNN
-	1    3650 3700
+P 3800 3500
+F 0 "R5" V 3800 3450 50  0000 L CNN
+F 1 "10K" V 3870 3455 50  0000 L CNN
+F 2 "Encoder:R_0603_1608Metric_Pad1.05x0.95mm_HandSolder" V 3730 3500 50  0001 C CNN
+F 3 "~" H 3800 3500 50  0001 C CNN
+	1    3800 3500
 	-1   0    0    1
 $EndComp
 Wire Wire Line
-	3800 4100 3800 3850
+	3800 4100 3800 3650
 Text Label 3500 6950 1    50   ~ 0
 2SIN+
@@
 	1    0    0    -1
 $EndComp
-Text Label 5500 6250 0    50   ~ 0
-USART3RX
-Text Label 6200 6250 2    50   ~ 0
+Text Label 5500 5200 0    50   ~ 0
+USART1RX
+Text Label 6200 5200 2    50   ~ 0
 BLETX
 Wire Wire Line
-	5450 6250 6250 6250
-Text Label 4700 7050 1    50   ~ 0
-USART3TX
-Text Label 4700 7350 1    50   ~ 0
+	5450 5200 6250 5200
+Text Label 4100 3700 3    50   ~ 0
+USART1TX
+Text Label 4100 3400 3    50   ~ 0
 BLERX
 Wire Wire Line
@@
 Wire Wire Line
 	3950 3300 3950 4000
-Wire Wire Line
-	3800 3850 3650 3850
 Text Label 3950 3500 1    50   ~ 0
 SIGB
@@
 Text Label 6200 5500 2    50   ~ 0
 OLEDSDA
-NoConn ~ 3650 4100
 NoConn ~ 4400 4100
 NoConn ~ 2850 4750
@@
 NoConn ~ 5450 5800
 NoConn ~ 5450 5650
-NoConn ~ 5450 5200
 NoConn ~ 5450 5050
 NoConn ~ 5450 4900
@@
 $EndComp
 Wire Wire Line
-	4100 4100 4100 3300
-Text Label 4100 3650 3    50   ~ 0
+	3650 4100 3650 3300
+Text Label 3650 3650 3    50   ~ 0
 EncEnable
 $Comp
@@
 	4550 6650 4550 7250
 Wire Wire Line
-	4700 6650 4700 7600
+	4100 4100 4100 3300
 $Comp
 L Encoder:STM32G431CBT6 U1
@@
 $EndComp
 NoConn ~ 2850 5050
+NoConn ~ 4700 6650
+NoConn ~ 5450 6250
 $EndSCHEMATC

Commit message: Advances
Parts:
- added C19, C20, C21, C22, C23, C24, C25, C26: 3.2uF, Encoder:C_0603_1608Metric_Pad1.05x0.95mm_HandSolder, symbol Device:C
- added R11, R12, R13, R14, R15, R16, R17, R18: 100, Encoder:R_0603_1608Metric_Pad1.05x0.95mm_HandSolder, symbol Device:R
Connections:
- wire segments 99 -> 107
Other:
- moved on the sheet: C1, C10, C11, C2, C3, C4, C5, C6, C7, C8, C9, J1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

Commit message: Changes
Changed lines of the file:
@@
 U 1 1 5EFA1FD1
 P 3400 5500
-F 0 "C4" V 3200 5450 50  0000 C CNN
-F 1 "100nF" V 3350 5300 50  0000 C CNN
+F 0 "C4" V 3350 5350 50  0000 C CNN
+F 1 "100nF" V 3350 5150 50  0000 C CNN
 F 2 "Encoder:C_0603_1608Metric_Pad1.05x0.95mm_HandSolder" H 3438 5350 50  0001 C CNN
 F 3 "~" H 3400 5500 50  0001 C CNN
@@
 NoConn ~ 3550 6250
 NoConn ~ 5100 6650
-NoConn ~ 6150 6100
 NoConn ~ 6150 5050
 NoConn ~ 6150 4900
@@
 	-1   0    0    1
 $EndComp
+NoConn ~ 4500 6650
+NoConn ~ 4650 6650
+Text GLabel 6150 6100 2    50   Input ~ 0
+CHG
+NoConn ~ 6150 5650
 Wire Wire Line
 	4050 6650 4050 7050
@@
 	1    0    0    -1
 $EndComp
-NoConn ~ 4500 6650
-NoConn ~ 4650 6650
-Text GLabel 6150 5950 2    50   Input ~ 0
-CHG
-NoConn ~ 6150 5650
+NoConn ~ 6150 5950
 $EndSCHEMATC

Commit message: Finished PCB
Parts:
- added R19, R20: 10K, Encoder:R_0603_1608Metric_Pad1.05x0.95mm_HandSolder, symbol Device:R
Connections:
- net labels added: VCC
- net labels removed: CHG
- wire segments 107 -> 108
Other:
- note added: "*Config as digital\ninput always!!\n"
Changed lines of the file:
@@
 Wire Wire Line
 	3150 4500 3150 4550
-Text GLabel 6150 5800 2    50   Input ~ 0
+Text GLabel 7650 5500 1    50   Input ~ 0
 Batt+
 Connection ~ 4950 7250
@@
 U 1 1 5F04A231
 P 1400 7100
-F 0 "R11" V 1350 6950 50  0000 C CNN
+F 0 "R11" V 1350 6900 50  0000 C CNN
 F 1 "100" V 1400 7100 50  0000 C CNN
 F 2 "Encoder:R_0603_1608Metric_Pad1.05x0.95mm_HandSolder" V 1330 7100 50  0001 C CNN
@@
 U 1 1 5F04DC3F
 P 1400 7200
-F 0 "R12" V 1350 7050 50  0000 C CNN
+F 0 "R12" V 1350 7000 50  0000 C CNN
 F 1 "100" V 1400 7200 50  0000 C CNN
 F 2 "Encoder:R_0603_1608Metric_Pad1.05x0.95mm_HandSolder" V 1330 7200 50  0001 C CNN
@@
 U 1 1 5F04DE20
 P 1400 7300
-F 0 "R13" V 1350 7150 50  0000 C CNN
+F 0 "R13" V 1350 7100 50  0000 C CNN
 F 1 "100" V 1400 7300 50  0000 C CNN
 F 2 "Encoder:R_0603_1608Metric_Pad1.05x0.95mm_HandSolder" V 1330 7300 50  0001 C CNN
@@
 U 1 1 5F04DF97
 P 1400 7400
-F 0 "R14" V 1350 7250 50  0000 C CNN
+F 0 "R14" V 1350 7200 50  0000 C CNN
 F 1 "100" V 1400 7400 50  0000 C CNN
 F 2 "Encoder:R_0603_1608Metric_Pad1.05x0.95mm_HandSolder" V 1330 7400 50  0001 C CNN
@@
 U 1 1 5F04E059
 P 1400 7500
-F 0 "R15" V 1350 7350 50  0000 C CNN
+F 0 "R15" V 1350 7300 50  0000 C CNN
 F 1 "100" V 1400 7500 50  0000 C CNN
 F 2 "Encoder:R_0603_1608Metric_Pad1.05x0.95mm_HandSolder" V 1330 7500 50  0001 C CNN
@@
 U 1 1 5F04E1B1
 P 1400 7600
-F 0 "R16" V 1350 7450 50  0000 C CNN
+F 0 "R16" V 1350 7400 50  0000 C CNN
 F 1 "100" V 1400 7600 50  0000 C CNN
 F 2 "Encoder:R_0603_1608Metric_Pad1.05x0.95mm_HandSolder" V 1330 7600 50  0001 C CNN
@@
 U 1 1 5F04E323
 P 1400 7700
-F 0 "R17" V 1350 7550 50  0000 C CNN
+F 0 "R17" V 1350 7500 50  0000 C CNN
 F 1 "100" V 1400 7700 50  0000 C CNN
 F 2 "Encoder:R_0603_1608Metric_Pad1.05x0.95mm_HandSolder" V 1330 7700 50  0001 C CNN
@@
 U 1 1 5F04E45C
 P 1400 7800
-F 0 "R18" V 1350 7650 50  0000 C CNN
+F 0 "R18" V 1350 7600 50  0000 C CNN
 F 1 "100" V 1400 7800 50  0000 C CNN
 F 2 "Encoder:R_0603_1608Metric_Pad1.05x0.95mm_HandSolder" V 1330 7800 50  0001 C CNN
@@
 NoConn ~ 4650 6650
 Text GLabel 6150 6100 2    50   Input ~ 0
-CHG
+VCC
 NoConn ~ 6150 5650
 Wire Wire Line
@@
 $EndComp
 NoConn ~ 6150 5950
+$Comp
+L Device:R R19
+U 1 1 5F0F6150
+P 7650 5650
+F 0 "R19" H 7720 5696 50  0000 L CNN
+F 1 "10K" H 7720 5605 50  0000 L CNN
+F 2 "Encoder:R_0603_1608Metric_Pad1.05x0.95mm_HandSolder" V 7580 5650 50  0001 C CNN
+F 3 "~" H 7650 5650 50  0001 C CNN
+	1    7650 5650
+	1    0    0    -1
+$EndComp
+$Comp
+L Device:R R20
+U 1 1 5F0F6BEE
+P 7650 5950
+F 0 "R20" H 7720 5996 50  0000 L CNN
+F 1 "10K" H 7720 5905 50  0000 L CNN
+F 2 "Encoder:R_0603_1608Metric_Pad1.05x0.95mm_HandSolder" V 7580 5950 50  0001 C CNN
+F 3 "~" H 7650 5950 50  0001 C CNN
+	1    7650 5950
+	1    0    0    -1
+$EndComp
+Connection ~ 7650 5800
+$Comp
+L power:GND #PWR0105
+U 1 1 5F0FACD0
+P 7650 6100
+F 0 "#PWR0105" H 7650 5850 50  0001 C CNN
+F 1 "GND" H 7655 5927 50  0000 C CNN
+F 2 "" H 7650 6100 50  0001 C CNN
+F 3 "" H 7650 6100 50  0001 C CNN
+	1    7650 6100
+	1    0    0    -1
+$EndComp
+Text Notes 6350 6150 0    50   ~ 0
+*Config as digital\ninput always!!\n
+Wire Wire Line
+	6150 5800 7650 5800
 $EndSCHEMATC

Commit message: Changes
Parts:
- added J6: Conn_01x04_Male, Encoder:PinHeader_2x02_P2.54mm_Vertical, symbol Connector:Conn_01x04_Male
Connections:
- wire segments 108 -> 116
Changed lines of the file:
@@
 Wire Wire Line
 	6150 5800 7650 5800
+$Comp
+L Connector:Conn_01x04_Male J6
+U 1 1 5F087510
+P 6550 2950
+F 0 "J6" V 6612 3094 50  0000 L CNN
+F 1 "Conn_01x04_Male" V 6703 3094 50  0000 L CNN
+F 2 "Encoder:PinHeader_2x02_P2.54mm_Vertical" H 6550 2950 50  0001 C CNN
+F 3 "~" H 6550 2950 50  0001 C CNN
+	1    6550 2950
+	0    1    1    0
+$EndComp
+$Comp
+L power:+3.3V #PWR011
+U 1 1 5F088CE6
+P 6400 3300
+F 0 "#PWR011" H 6400 3150 50  0001 C CNN
+F 1 "+3.3V" V 6400 3550 50  0000 C CNN
+F 2 "" H 6400 3300 50  0001 C CNN
+F 3 "" H 6400 3300 50  0001 C CNN
+	1    6400 3300
+	-1   0    0    1
+$EndComp
+$Comp
+L power:GND #PWR012
+U 1 1 5F08ACC7
+P 6600 3300
+F 0 "#PWR012" H 6600 3050 50  0001 C CNN
+F 1 "GND" V 6600 3100 50  0000 C CNN
+F 2 "" H 6600 3300 50  0001 C CNN
+F 3 "" H 6600 3300 50  0001 C CNN
+	1    6600 3300
+	1    0    0    -1
+$EndComp
+Wire Wire Line
+	6600 3300 6550 3300
+Wire Wire Line
+	6550 3300 6550 3150
+Wire Wire Line
+	6600 3300 6650 3300
+Wire Wire Line
+	6650 3300 6650 3150
+Connection ~ 6600 3300
+Wire Wire Line
+	6400 3300 6350 3300
+Wire Wire Line
+	6350 3300 6350 3150
+Wire Wire Line
+	6400 3300 6450 3300
+Wire Wire Line
+	6450 3300 6450 3150
+Connection ~ 6400 3300
 $EndSCHEMATC

Commit message: Schematic change
Changed lines of the file:
@@
 L power:+3.3V #PWR0104
 U 1 1 5EFE29C0
-P 3150 3850
-F 0 "#PWR0104" H 3150 3700 50  0001 C CNN
-F 1 "+3.3V" H 3165 4023 50  0000 C CNN
-F 2 "" H 3150 3850 50  0001 C CNN
-F 3 "" H 3150 3850 50  0001 C CNN
-	1    3150 3850
-	1    0    0    -1
-$EndComp
-Wire Wire Line
-	3150 4150 3150 4500
-Text Label 3150 4150 3    50   ~ 0
-Supply
+P 3150 3450
+F 0 "#PWR0104" H 3150 3300 50  0001 C CNN
+F 1 "+3.3V" H 3165 3623 50  0000 C CNN
+F 2 "" H 3150 3450 50  0001 C CNN
+F 3 "" H 3150 3450 50  0001 C CNN
+	1    3150 3450
+	1    0    0    -1
+$EndComp
 Wire Wire Line
 	6300 4600 6300 4100
@@
 Text Label 6300 4250 3    50   ~ 0
 Supply
-Text Label 4050 3700 3    50   ~ 0
+Text Label 3150 3550 3    50   ~ 0
 Supply
 $Comp
@@
 Text Label 4350 3650 3    50   ~ 0
 EncEnable
-$Comp
-L power:PWR_FLAG #FLG0102
-U 1 1 5EFDA81C
-P 3150 4500
-F 0 "#FLG0102" H 3150 4575 50  0001 C CNN
-F 1 "PWR_FLAG" V 3150 4627 50  0000 L CNN
-F 2 "" H 3150 4500 50  0001 C CNN
-F 3 "~" H 3150 4500 50  0001 C CNN
-	1    3150 4500
-	0    -1   -1   0
-$EndComp
-Connection ~ 3150 4500
-Wire Wire Line
-	3150 4500 3150 4550
 Text GLabel 7650 5500 1    50   Input ~ 0
 Batt+
@@
 	6450 3300 6450 3150
 Connection ~ 6400 3300
+Wire Wire Line
+	3150 4150 3150 4200
+$Comp
+L power:GND #PWR0106
+U 1 1 5F0AE8F0
+P 3150 4200
+F 0 "#PWR0106" H 3150 3950 50  0001 C CNN
+F 1 "GND" H 3155 4027 50  0000 C CNN
+F 2 "" H 3150 4200 50  0001 C CNN
+F 3 "" H 3150 4200 50  0001 C CNN
+	1    3150 4200
+	1    0    0    -1
+$EndComp
+Wire Wire Line
+	3150 3450 3150 3850
+Text Label 4050 3600 3    50   ~ 0
+Supply
 $EndSCHEMATC
