File: Mechatronics/Hardware/Electrical/BSensorsBoard/SensorsBoard.kicad_pcb (KiCad board)
At the start: 2 copper layers, 9.4 x 40.7 mm, 10 parts, among them J1 Conn_01x01_Male, J2 Conn_01x01_Male, J3 Conn_01x01_Male, J4 Conn_01x01_Male, U1 ITR1802

Commit message: Changes
Parts:
- U8 (x2): renamed from U1; value ITR1802 -> ITR8102
Connections:
- J1 pad 1: (no net) -> Net-(J1-Pad1)
- J2 pad 1: (no net) -> Net-(J2-Pad1)
- J3 pad 1: (no net) -> Net-(J3-Pad1)
- J4 pad 1: (no net) -> Net-(J4-Pad1)
- U8 pad 1: (no net) -> Net-(J1-Pad1)
- U8 pad 2: (no net) -> Net-(J2-Pad1)
- U8 pad 3: (no net) -> Net-(J4-Pad1)
- U8 pad 4: (no net) -> Net-(J3-Pad1)
Routing:
- net (no net): track 36.6 -> 0.00 mm
- net Net-(J2-Pad1): track 9.79 -> 19.6 mm
- net Net-(J1-Pad1): track 9.53 -> 19.1 mm
- net Net-(J4-Pad1): track 8.81 -> 17.6 mm
- net Net-(J3-Pad1): track 8.42 -> 16.8 mm
