File: Mechatronics/Hardware/Electrical/BEncoderBoard2/EncoderBoard2.kicad_pcb (KiCad board)
At the start: 2 copper layers, 37.8 x 59.2 mm, 66 parts, among them IC1 TP4056, IC2 DW01+G, J1 MagSensors_Conn, J2 OLED/SWD_Conn, J3 Barrel_Jack_Switch, J4 GNDPWR, J5 Batt_Conn, J6 MagSensors_Power, Q1 DMosfet, Q2 Q_PMOS_GSD, Q3 Q_PMOS_GSD, U1 STM32G431CBT6, U2 OPTO_Conn, U3 OPTO_Conn, U4 RN4871, U5 82402305, U6 LTC3240, Y1 8Mhz

Commit message: PCB changes
Connections:
- IC1 pad 9: Net-(IC1-Pad9) -> GND
Routing:
- net GND: track 78.3 -> 82.1 mm, vias 39 -> 60
- added copper zone on F.Cu, net GND
