File: Mechatronics/Hardware/Electrical/BEncoderBoard3(1.2)/EncoderBoard3(1.2).kicad_pcb (KiCad board)
At the start: 2 copper layers, 24.6 x 68.1 mm, 51 parts, among them J1 Conn_01x08_Male, J2 Conn_01x03_Male, J3 Conn_01x04_Male, J4 Conn_01x04_Male, J6 Conn_01x06_Male, J7 Conn_01x03_Male, J8 Conn_01x02_Male, P1 TYPE-C-31-M-12, Q1 Q_PMOS_GSD, Q2 Q_PMOS_GSD, U1 STM32G431KBT6, U3 LTC3240, U4 82402305, U5 DW01+G, U6 DMosfet, U7 TP4056, Y1 8Mhz

Commit message: PCB changes
Parts:
- removed the C3 at (126.5, 90.5)
- added C5: 12pF, Encoder:C_0603_1608Metric_Pad1.05x0.95mm_HandSolder, F.Cu at (126.5, 90.5)
- H1, H2: renamed from REF**; value MountingHole_3.2mm_M3_Pad -> MountingHole_Pad
- J1: moved to F.Cu
- moved J1 17.4 mm to (139.8, 92.0), turned to 270 degrees
- moved C15 2.08 mm to (127.7, 137.1)
- moved H1 1.05 mm to (125.0, 142.4)
- moved P1 1.00 mm to (136.3, 148.5)
- renumbered C9 to C1, C8 to C10, C13 to C11, C14 to C12, C15 to C13, C16 to C14, C17 to C15, C10 to C2, C1 to C3, C2 to C4, C5 to C6, C6 to C7, C4 to C8, C7 to C9, R16 to R15, R15 to R16, R6 to R3, R3 to R4, R7 to R5, R4 to R6, R5 to R7, R9 to R8, R8 to R9
Connections:
- H1 pad 1: (no net) -> GND
- H2 pad 1: (no net) -> GND
- J1 pad 1: /E+(a) -> /D+(a)
- J1 pad 2: /E-(b) -> GND
- J1 pad 3: GND -> /E-(a)
- J1 pad 4: /D+(b) -> /E+(a)
- J1 pad 5: /E+(a) -> /D+(b)
- J1 pad 6: /E-(a) -> GND
- J1 pad 7: GND -> /E-(b)
- J1 pad 8: /D+(a) -> /E+(a)
Routing:
- net GND: track 56.8 -> 54.4 mm
- net VCC: track 105.7 -> 106.8 mm
- net Net-(P1-PadB5): track 2.40 -> 3.41 mm
- net Net-(P1-PadA5): track 6.24 -> 7.24 mm
Other:
- board size 24.6 x 68.1 mm -> 24.6 x 69.1 mm
- board text added: "-"
- board text added: "D"
- board text added: "E"
