File: Mechatronics/Hardware/Electrical/BEncoderBoard3(1.2)/Power.sch (KiCad schematic (older format))
At the start: 22 parts, among them J7 Conn_01x03_Male, J8 Conn_01x02_Male, P1 TYPE-C-31-M-12, Q2 Q_PMOS_GSD, U3 LTC3240, U4 82402305, U5 DW01+G, U6 DMosfet, U7 TP4056

Commit message: PCB changes
Parts:
- R10: value 5.1k -> 5.1K
- renumbered C13 to C11, C14 to C12, C15 to C13, C16 to C14, C17 to C15, R16 to R15, R15 to R16
Changed lines of the file:
@@
 P 7650 2950
 AR Path="/5F137029" Ref="R?"  Part="1"
-AR Path="/5F11DB77/5F137029" Ref="R16"  Part="1"
-F 0 "R16" H 7720 2996 50  0000 L CNN
+AR Path="/5F11DB77/5F137029" Ref="R15"  Part="1"
+F 0 "R15" H 7720 2996 50  0000 L CNN
 F 1 "10K" H 7720 2905 50  0000 L CNN
 F 2 "Encoder:R_0603_1608Metric_Pad1.05x0.95mm_HandSolder" V 7580 2950 50  0001 C CNN
@@
 P 10150 3850
 AR Path="/5F137035" Ref="C?"  Part="1"
-AR Path="/5F11DB77/5F137035" Ref="C15"  Part="1"
-F 0 "C15" H 10265 3896 50  0000 L CNN
+AR Path="/5F11DB77/5F137035" Ref="C13"  Part="1"
+F 0 "C13" H 10265 3896 50  0000 L CNN
 F 1 "1uF" H 10265 3805 50  0000 L CNN
 F 2 "Encoder:C_0603_1608Metric_Pad1.05x0.95mm_HandSolder" H 10188 3700 50  0001 C CNN
@@
 P 8300 3600
 AR Path="/5F137041" Ref="C?"  Part="1"
-AR Path="/5F11DB77/5F137041" Ref="C14"  Part="1"
-F 0 "C14" H 8415 3646 50  0000 L CNN
+AR Path="/5F11DB77/5F137041" Ref="C12"  Part="1"
+F 0 "C12" H 8415 3646 50  0000 L CNN
 F 1 "1uF" H 8415 3555 50  0000 L CNN
 F 2 "Encoder:C_0603_1608Metric_Pad1.05x0.95mm_HandSolder" H 8338 3450 50  0001 C CNN
@@
 P 8300 4100
 AR Path="/5F137047" Ref="C?"  Part="1"
-AR Path="/5F11DB77/5F137047" Ref="C13"  Part="1"
-F 0 "C13" H 8415 4146 50  0000 L CNN
+AR Path="/5F11DB77/5F137047" Ref="C11"  Part="1"
+F 0 "C11" H 8415 4146 50  0000 L CNN
 F 1 "4.7uF" H 8415 4055 50  0000 L CNN
 F 2 "Encoder:C_0603_1608Metric_Pad1.05x0.95mm_HandSolder" H 8338 3950 50  0001 C CNN
@@
 P 4050 4100
 AR Path="/5F137077" Ref="R?"  Part="1"
-AR Path="/5F11DB77/5F137077" Ref="R15"  Part="1"
-F 0 "R15" H 3800 4150 50  0000 L CNN
+AR Path="/5F11DB77/5F137077" Ref="R16"  Part="1"
+F 0 "R16" H 3800 4150 50  0000 L CNN
 F 1 "1.5K" H 3750 4050 50  0000 L CNN
 F 2 "Encoder:R_0603_1608Metric_Pad1.05x0.95mm_HandSolder" V 3980 4100 50  0001 C CNN
@@
 P 3400 2950
 AR Path="/5F137083" Ref="C?"  Part="1"
-AR Path="/5F11DB77/5F137083" Ref="C17"  Part="1"
-F 0 "C17" H 3515 2996 50  0000 L CNN
+AR Path="/5F11DB77/5F137083" Ref="C15"  Part="1"
+F 0 "C15" H 3515 2996 50  0000 L CNN
 F 1 "10uF" H 3515 2905 50  0000 L CNN
 F 2 "Encoder:C_0603_1608Metric_Pad1.05x0.95mm_HandSolder" H 3438 2800 50  0001 C CNN
@@
 P 6000 4500
 AR Path="/5F1370A8" Ref="C?"  Part="1"
-AR Path="/5F11DB77/5F1370A8" Ref="C16"  Part="1"
-F 0 "C16" H 6115 4546 50  0000 L CNN
+AR Path="/5F11DB77/5F1370A8" Ref="C14"  Part="1"
+F 0 "C14" H 6115 4546 50  0000 L CNN
 F 1 "100nF" H 6115 4455 50  0000 L CNN
 F 2 "Encoder:C_0603_1608Metric_Pad1.05x0.95mm_HandSolder" H 6038 4350 50  0001 C CNN
@@
 P 3000 3300
 F 0 "R10" H 3070 3346 50  0000 L CNN
-F 1 "5.1k" H 3070 3255 50  0000 L CNN
+F 1 "5.1K" H 3070 3255 50  0000 L CNN
 F 2 "Encoder:R_0603_1608Metric_Pad1.05x0.95mm_HandSolder" V 2930 3300 50  0001 C CNN
 F 3 "~" H 3000 3300 50  0001 C CNN
