File: Mechatronics/Hardware/Electrical/BEncoderBoard3(2)/BEncoderBoard3(2).sch (KiCad schematic (older format))
At the start: 10 parts, among them J1 Conn_01x01_Male, J2 Conn_01x01_Male, J3 Conn_01x01_Male, J4 Conn_01x01_Male, J5 Conn_01x01_Male, J6 Conn_01x01_Male, J7 Conn_01x01_Male, J8 Conn_01x01_Male, Q3 ITR8102, Q4 ITR8102

Commit message: PCB changes
Parts:
- Q3, Q4: symbol SensorsBoard-rescue:ITR1802-Encoder -> Encoder:ITR8102
Changed lines of the file:
@@
 $EndDescr
 $Comp
-L SensorsBoard-rescue:ITR1802-Encoder Q3
+L Encoder:ITR8102 Q3
 U 1 1 5C59CA18
 P 5900 4500
@@
 	5350 4400 5600 4400
 $Comp
-L SensorsBoard-rescue:ITR1802-Encoder Q4
+L Encoder:ITR8102 Q4
 U 1 1 6081B0B0
 P 5900 5250
